File: hw/Altimeter/Altimeter.sch (EAGLE design)
At the start: 58 parts, among them U1 ATSAMD21G-A, U2 MPU-9250, U3 MS5803-14BA, X1 22-23-2041, X2 22-23-2041, Y1 32.768kHx

Commit message: dasAltimeter
Parts:
- added C16: 0.1uF, SparkFun-Passives:CAP0402-CAP
- added U$7: ADXL193, SparkFun-Sensors:ADXL193
Connections:
- new net ACCELX: U$7.OUT, U1.PA07(AIN7/SER0:3/TC1:1)
- net 3.3V: now also C16.1, U$7.VDD, U$7.VDD2
- net GND: now also C16.2, U$7.GND
Changed lines of the file:
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@@
 <?xml version="1.0" encoding="utf-8"?>
 <!DOCTYPE eagle SYSTEM "eagle.dtd">
-<eagle version="8.3.1">
+<eagle version="8.3.2">
 <drawing>
 <settings>
@@
 <part name="SUPPLY12" library="SparkFun-Aesthetics" deviceset="3.3V" device=""/>
 <part name="GND4" library="SparkFun-Aesthetics" deviceset="GND" device=""/>
+<part name="U$7" library="SparkFun-Sensors" deviceset="ADXL193" device=""/>
+<part name="GND52" library="SparkFun-Aesthetics" deviceset="GND" device=""/>
+<part name="SUPPLY23" library="SparkFun-Aesthetics" deviceset="3.3V" device=""/>
+<part name="GND53" library="SparkFun-Aesthetics" deviceset="GND" device=""/>
+<part name="C16" library="SparkFun-Passives" deviceset="CAP" device="0402-CAP" value="0.1uF"/>
 </parts>
 <sheets>
@@
 <instance part="SUPPLY12" gate="G$1" x="205.74" y="261.62"/>
 <instance part="GND4" gate="1" x="205.74" y="236.22"/>
+<instance part="U$7" gate="G$1" x="48.26" y="81.28"/>
+<instance part="GND52" gate="1" x="63.5" y="73.66"/>
+<instance part="SUPPLY23" gate="G$1" x="22.86" y="91.44"/>
+<instance part="GND53" gate="1" x="22.86" y="71.12"/>
+<instance part="C16" gate="G$1" x="22.86" y="78.74" smashed="yes">
+<attribute name="NAME" x="24.384" y="81.661" size="1.778" layer="95"/>
+<attribute name="VALUE" x="22.86" y="76.327" size="1.778" layer="96"/>
+</instance>
 </instances>
 <busses>
@@
 <pinref part="SUPPLY12" gate="G$1" pin="3.3V"/>
 <wire x1="205.74" y1="261.62" x2="205.74" y2="256.54" width="0.1524" layer="91"/>
+</segment>
+<segment>
+<pinref part="U$7" gate="G$1" pin="VDD2"/>
+<wire x1="22.86" y1="83.82" x2="30.48" y2="83.82" width="0.1524" layer="91"/>
+<wire x1="30.48" y1="83.82" x2="30.48" y2="81.28" width="0.1524" layer="91"/>
+<wire x1="30.48" y1="81.28" x2="35.56" y2="81.28" width="0.1524" layer="91"/>
+<pinref part="C16" gate="G$1" pin="1"/>
+<pinref part="U$7" gate="G$1" pin="VDD"/>
+<wire x1="35.56" y1="83.82" x2="30.48" y2="83.82" width="0.1524" layer="91"/>
+<junction x="30.48" y="83.82"/>
+<pinref part="SUPPLY23" gate="G$1" pin="3.3V"/>
+<wire x1="22.86" y1="83.82" x2="22.86" y2="91.44" width="0.1524" layer="91"/>
+<junction x="22.86" y="83.82"/>
 </segment>
 </net>
@@
 <wire x1="205.74" y1="238.76" x2="205.74" y2="243.84" width="0.1524" layer="91"/>
 </segment>
+<segment>
+<pinref part="C16" gate="G$1" pin="2"/>
+<pinref part="GND53" gate="1" pin="GND"/>
+<wire x1="22.86" y1="73.66" x2="22.86" y2="76.2" width="0.1524" layer="91"/>
+</segment>
+<segment>
+<pinref part="U$7" gate="G$1" pin="GND"/>
+<pinref part="GND52" gate="1" pin="GND"/>
+<wire x1="60.96" y1="78.74" x2="63.5" y2="78.74" width="0.1524" layer="91"/>
+<wire x1="63.5" y1="78.74" x2="63.5" y2="76.2" width="0.1524" layer="91"/>
+</segment>
 </net>
 <net name="N$3" class="0">
@@
 <pinref part="R13" gate="G$1" pin="2"/>
 <wire x1="25.4" y1="17.78" x2="22.86" y2="17.78" width="0.1524" layer="91"/>
-<wire x1="22.86" y1="17.78" x2="12.7" y2="17.78" width="0.1524" layer="91"/>
+<wire x1="22.86" y1="17.78" x2="10.16" y2="17.78" width="0.1524" layer="91"/>
 <junction x="22.86" y="17.78"/>
-<label x="12.7" y="17.78" size="1.27" layer="95" rot="R180" xref="yes"/>
+<label x="10.16" y="17.78" size="1.27" layer="95" rot="R180" xref="yes"/>
 <pinref part="S2" gate="G$1" pin="1"/>
 </segment>
@@
 <net name="FIRE_C" class="0">
 <segment>
-<wire x1="279.4" y1="48.26" x2="276.86" y2="48.26" width="0.1524" layer="91"/>
 <label x="271.78" y="48.26" size="1.27" layer="95" rot="R180" xref="yes"/>
 <pinref part="R5" gate="G$1" pin="2"/>
 <pinref part="R6" gate="G$1" pin="1"/>
 <junction x="279.4" y="48.26"/>
-<wire x1="276.86" y1="48.26" x2="271.78" y2="48.26" width="0.1524" layer="91"/>
-<wire x1="266.7" y1="57.15" x2="276.86" y2="57.15" width="0.1524" layer="91"/>
-<wire x1="276.86" y1="57.15" x2="276.86" y2="48.26" width="0.1524" layer="91"/>
-<junction x="276.86" y="48.26"/>
+<wire x1="279.4" y1="48.26" x2="271.78" y2="48.26" width="0.1524" layer="91"/>
 </segment>
 <segment>
@@
 <net name="FIRE_D" class="0">
 <segment>
-<wire x1="279.4" y1="25.4" x2="274.32" y2="25.4" width="0.1524" layer="91"/>
+<wire x1="279.4" y1="25.4" x2="271.78" y2="25.4" width="0.1524" layer="91"/>
 <label x="271.78" y="25.4" size="1.27" layer="95" rot="R180" xref="yes"/>
 <pinref part="R7" gate="G$1" pin="2"/>
 <pinref part="R8" gate="G$1" pin="1"/>
 <junction x="279.4" y="25.4"/>
-<wire x1="274.32" y1="25.4" x2="271.78" y2="25.4" width="0.1524" layer="91"/>
-<wire x1="266.7" y1="34.29" x2="274.32" y2="34.29" width="0.1524" layer="91"/>
-<wire x1="274.32" y1="34.29" x2="274.32" y2="25.4" width="0.1524" layer="91"/>
-<junction x="274.32" y="25.4"/>
 </segment>
 <segment>
@@
 </segment>
 </net>
+<net name="ACCELX" class="0">
+<segment>
+<pinref part="U$7" gate="G$1" pin="OUT"/>
+<wire x1="60.96" y1="83.82" x2="66.04" y2="83.82" width="0.1524" layer="91"/>
+<label x="66.04" y="83.82" size="1.27" layer="95" xref="yes"/>
+</segment>
+<segment>
+<pinref part="U1" gate="G$1" pin="PA07(AIN7/SER0:3/TC1:1)"/>
+<wire x1="172.72" y1="134.62" x2="170.18" y2="134.62" width="0.1524" layer="91"/>
+<label x="170.18" y="134.62" size="1.778" layer="95" rot="R180"/>
+</segment>
+</net>
 </nets>
 </sheet>
 </sheets>
+<errors>
+</errors>
 </schematic>
 </drawing>

Commit message: day one changes
Connections:
- net CS_IMU: now also U1.PA20(SER5:2+)
Changed lines of the file:
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@@
 <junction x="401.32" y="195.58"/>
+</segment>
+<segment>
+<pinref part="U1" gate="G$1" pin="PA20(SER5:2+)"/>
+<wire x1="241.3" y1="144.78" x2="243.84" y2="144.78" width="0.1524" layer="91"/>
+<label x="243.84" y="144.78" size="1.778" layer="95"/>
 </segment>
 </net>
