File: hw/DasAltimeter v1.1/DasAltimeter v1.1.brd (EAGLE design)
At the start: 49.1 x 20.6 mm, 57 parts, among them U1 ATSAMD21G-A, U2 MPU-9250, U3 MS5803-14BA, X1 22-23-2041, X2 22-23-2041, Y1 32.768kHx

Commit message: day one changes
Parts:
- moved JP1 0.36 mm to (31.0, 21.1), flipped to the bottom, turned to 180 degrees
Routing:
- net !RESET: track 11.0 -> 12.0 mm, vias 0 -> 1
- net SWCLK: track 12.5 -> 13.6 mm, vias 0 -> 1
- net SWDIO: track 11.3 -> 11.4 mm, vias 1 -> 2
Changed lines of the file:
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@@
 </element>
 <element name="FRAME1" library="SparkFun-Aesthetics" package="CREATIVE_COMMONS" value="FRAME-LEDGER" x="-80.01" y="22.86"/>
-<element name="JP1" library="SparkFun-Connectors" package="2X5-PTH-1.27MM" value="CORTEX_DEBUGPTH" x="31.242" y="20.828" smashed="yes"/>
+<element name="JP1" library="SparkFun-Connectors" package="2X5-PTH-1.27MM" value="CORTEX_DEBUGPTH" x="30.988" y="21.082" smashed="yes" rot="MR180"/>
 <element name="L1" library="SparkFun-Passives" package="0603" value="FB - 30Ohm" x="24.003" y="4.572" smashed="yes" rot="R90">
 <attribute name="NAME" x="24.13" y="6.223" size="0.4064" layer="25" font="vector" rot="R90"/>
@@
 <wire x1="47.625" y1="8.763" x2="47.736" y2="10.948" width="0" layer="19" extent="1-15"/>
 <wire x1="39.545" y1="18.923" x2="41.798" y2="13.97" width="0" layer="19" extent="1-1"/>
-<wire x1="28.702" y1="20.193" x2="32.810659375" y2="17.649746875" width="0" layer="19" extent="1-1"/>
-<wire x1="27.00261875" y1="16.685378125" x2="28.702" y2="20.193" width="0" layer="19" extent="1-1"/>
+<wire x1="28.448" y1="21.717" x2="32.810659375" y2="17.649746875" width="0" layer="19" extent="1-1"/>
+<wire x1="27.00261875" y1="16.685378125" x2="28.448" y2="21.717" width="0" layer="19" extent="1-1"/>
 <wire x1="23.2711" y1="16.5791" x2="26.67" y2="16.51" width="0" layer="19" extent="1-1"/>
 <wire x1="37.724" y1="9.134" x2="41.798" y2="13.97" width="0" layer="19" extent="1-16"/>
@@
 <wire x1="23.114" y1="18.376" x2="26.083378125" y2="17.955378125" width="0" layer="19" extent="1-1"/>
 <wire x1="23.296" y1="20.955" x2="23.114" y2="18.376" width="0" layer="19" extent="1-1"/>
-<wire x1="29.972" y1="20.193" x2="26.972378125" y2="18.36661875" width="0" layer="19" extent="1-1"/>
-<wire x1="31.242" y1="20.193" x2="29.972" y2="20.193" width="0" layer="19" extent="1-1"/>
-<wire x1="33.1642125" y1="17.29619375" x2="31.242" y2="20.193" width="0" layer="19" extent="1-1"/>
+<wire x1="29.718" y1="21.717" x2="26.972378125" y2="18.36661875" width="0" layer="19" extent="1-1"/>
+<wire x1="30.988" y1="21.717" x2="29.718" y2="21.717" width="0" layer="19" extent="1-1"/>
+<wire x1="33.1642125" y1="17.29619375" x2="30.988" y2="21.717" width="0" layer="19" extent="1-1"/>
 <wire x1="28.214465625" y1="10.225125" x2="31.369" y2="12.319" width="0" layer="19" extent="1-1"/>
 <wire x1="27.051" y1="9.398" x2="28.214465625" y2="10.225125" width="0" layer="19" extent="1-1"/>
@@
 <contactref element="R1" pad="1"/>
 <contactref element="JP1" pad="10"/>
-<wire x1="33.782" y1="21.463" x2="33.797" y2="21.478" width="0.254" layer="1"/>
+<wire x1="33.528" y1="20.447" x2="33.797" y2="21.478" width="0.254" layer="16"/>
 <wire x1="34.67465" y1="21.478" x2="33.797" y2="21.478" width="0.254" layer="1"/>
 <wire x1="34.67465" y1="21.478" x2="35.433" y2="21.478" width="0.254" layer="1"/>
@@
 <wire x1="34.163" y1="19.177" x2="34.67465" y2="19.68865" width="0.254" layer="1"/>
 <wire x1="34.67465" y1="19.68865" x2="34.67465" y2="21.478" width="0.254" layer="1"/>
+<via x="33.797" y="21.478" extent="1-16" drill="0.35"/>
 </signal>
 <signal name="N$5">
@@
 <via x="26.797" y="21.336" extent="1-16" drill="0.35"/>
 <wire x1="26.797" y1="21.336" x2="26.924" y2="21.463" width="0.254" layer="16"/>
-<wire x1="26.924" y1="21.463" x2="28.702" y2="21.463" width="0.254" layer="16"/>
+<wire x1="26.924" y1="21.463" x2="28.448" y2="20.447" width="0.254" layer="1"/>
 <wire x1="26.797" y1="20.32" x2="26.797" y2="21.336" width="0.254" layer="1"/>
+<via x="26.924" y="21.463" extent="1-16" drill="0.35"/>
 </signal>
 <signal name="SWCLK">
@@
 <wire x1="27.813" y1="22.225" x2="29.337" y2="22.225" width="0.254" layer="1"/>
 <wire x1="29.337" y1="22.225" x2="29.972" y2="21.59" width="0.254" layer="1"/>
-<wire x1="29.972" y1="21.59" x2="29.972" y2="21.463" width="0.254" layer="1"/>
+<wire x1="29.972" y1="21.59" x2="29.718" y2="20.447" width="0.254" layer="16"/>
+<via x="29.972" y="21.59" extent="1-16" drill="0.35"/>
 </signal>
 <signal name="CS_MEM">

Commit message: dasaltimeter 1.1 board work
Parts:
- moved C13 25.0 mm to (26.3, 2.54)
- moved D2 19.7 mm to (38.4, 8.38), turned to 270 degrees
- moved R23 19.6 mm to (38.4, 7.75), turned to 90 degrees
- moved U2 19.1 mm to (29.0, 2.54), turned to 0 degrees
- moved C12 18.3 mm to (31.6, 2.41), turned to 90 degrees
- moved R28 18.1 mm to (28.4, 6.48)
- moved U$7 17.9 mm to (22.9, 2.79), turned to 90 degrees
- moved STANDOFF3 13.8 mm to (36.6, 2.92)
- moved SG1 13.4 mm to (33.8, 15.6), turned to 180 degrees
- moved C9 12.5 mm to (35.1, 16.8), turned to 90 degrees
- moved C8 12.0 mm to (25.9, 16.3), turned to 315 degrees
- moved MEM 11.1 mm to (31.5, 17.7), turned to 270 degrees
- moved C16 10.9 mm to (26.0, 3.68), turned to 270 degrees
- moved C1 9.49 mm to (16.4, 19.4), turned to 270 degrees
- moved C4 9.30 mm to (18.4, 15.6)
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Routing:
- net RAW: track 59.1 -> 0.00 mm, vias 2 -> 0
- net 3.3V: track 59.0 -> 0.00 mm, vias 8 -> 0
- net FIRE_A: track 24.8 -> 0.00 mm, vias 2 -> 0
- net SENSE_D: track 23.7 -> 0.00 mm, vias 2 -> 0
- net GND: track 22.7 -> 0.00 mm, vias 17 -> 0
- net SENSE_A: track 20.8 -> 0.00 mm, vias 2 -> 0
- net FIRE_D: track 20.7 -> 0.00 mm, vias 2 -> 0
- net FIRE_B: track 19.4 -> 0.00 mm, vias 2 -> 0
- net CS_IMU: track 19.0 -> 0.00 mm, vias 2 -> 0
- net SPI1_MISO: track 18.9 -> 0.00 mm
- net SPI1_SCK: track 18.1 -> 0.00 mm
- net SENSE_C: track 15.1 -> 0.00 mm, vias 2 -> 0
- net FIRE_C: track 14.4 -> 0.00 mm, vias 2 -> 0
- net CS_MEM: track 14.4 -> 0.00 mm
- net BUZZER: track 14.3 -> 0.00 mm, vias 1 -> 0
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Other:
- board size 49.1 x 20.6 mm -> 39.4 x 21.8 mm

Commit message: changes to eagle stuff
Parts:
- R10, R12, R16, R22: value 27K -> (none); device SparkFun-Resistors:0402-RES -> SparkFun-Resistors:0402
- R11, R15, R21, R9: value 100K -> (none); device SparkFun-Resistors:0402-RES -> SparkFun-Resistors:0402
- R14, R17, R6, R7: value 100 -> (none); device SparkFun-Resistors:0402-RES -> SparkFun-Resistors:0402
- R20, R4, R5, R8: value 3.3k -> (none); device SparkFun-Resistors:0402-RES -> SparkFun-Resistors:0402
- R23: value 63 -> (none); device SparkFun-Resistors:0402-RES -> SparkFun-Resistors:0402

Commit message: DasAltimeter V0.1 board layout done
Parts:
- JP1: value CORTEX_DEBUGPTH -> CORTEX_DEBUG_PTH
- SG1: value BUZZERSMD2 -> BUZZER-SMD_KIT; device SparkFun-Electromechanical:BUZZER-CCV -> SparkFun-Electromechanical:BUZZER-CCV-KIT
- U$7: device SparkFun-Sensors:ADXL193 -> SparkFun-Sensors:LCC-8
