File: hw/DasAltimeter v1.1/DasAltimeter v1.1.sch (EAGLE design)
At the start: 60 parts, among them U1 ATSAMD21G-A, U2 MPU-9250, U3 MS5803-14BA, X1 22-23-2041, X2 22-23-2041, Y1 32.768kHx

Commit message: minor v1.1 borad changes
Parts:
- removed R13: 10k, SparkFun-Passives:RESISTOR0402-RES
- removed S2: SWITCH-MOMENTARY-2SMD-4.6X2.8MM, SparkFun-Electromechanical:SWITCH-MOMENTARY-2SMD-4.6X2.8MM
Connections:
- net 3.3V: no longer S2.2
- net GND: no longer R13.1
- net PROG: no longer R13.2, S2.1
Changed lines of the file:
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@@
 <part name="SUPPLY6" library="SparkFun-Aesthetics" deviceset="3.3V" device=""/>
 <part name="GND11" library="SparkFun-Aesthetics" deviceset="GND" device=""/>
-<part name="R13" library="SparkFun-Passives" deviceset="RESISTOR" device="0402-RES" value="10k"/>
-<part name="SUPPLY13" library="SparkFun-Aesthetics" deviceset="3.3V" device=""/>
-<part name="GND21" library="SparkFun-Aesthetics" deviceset="GND" device=""/>
-<part name="S2" library="SparkFun-Electromechanical" deviceset="SWITCH-MOMENTARY-2" device="SMD-4.6X2.8MM"/>
 <part name="MEM" library="SaL-lib" deviceset="AT25SF081" device=""/>
 <part name="C9" library="SparkFun-Passives" deviceset="CAP" device="0402-CAP" value="0.1uF"/>
@@
 <instance part="SUPPLY6" gate="G$1" x="7.62" y="53.34"/>
 <instance part="GND11" gate="1" x="7.62" y="35.56"/>
-<instance part="R13" gate="G$1" x="22.86" y="12.7" rot="R90"/>
-<instance part="SUPPLY13" gate="G$1" x="40.64" y="17.78"/>
-<instance part="GND21" gate="1" x="22.86" y="5.08"/>
-<instance part="S2" gate="G$1" x="30.48" y="17.78"/>
 <instance part="MEM" gate="G$1" x="375.92" y="88.9"/>
 <instance part="C9" gate="G$1" x="363.22" y="81.28" smashed="yes">
@@
 </segment>
 <segment>
-<pinref part="SUPPLY13" gate="G$1" pin="3.3V"/>
-<wire x1="35.56" y1="17.78" x2="40.64" y2="17.78" width="0.1524" layer="91"/>
-<pinref part="S2" gate="G$1" pin="2"/>
-</segment>
-<segment>
 <pinref part="MEM" gate="G$1" pin="!WP"/>
 <wire x1="373.38" y1="81.28" x2="370.84" y2="81.28" width="0.1524" layer="91" style="longdash"/>
@@
 </segment>
 <segment>
-<pinref part="R13" gate="G$1" pin="1"/>
-<pinref part="GND21" gate="1" pin="GND"/>
-</segment>
-<segment>
 <pinref part="MEM" gate="G$1" pin="GND"/>
 <pinref part="C9" gate="G$1" pin="2"/>
@@
 <net name="PROG" class="0">
 <segment>
-<pinref part="R13" gate="G$1" pin="2"/>
-<wire x1="25.4" y1="17.78" x2="22.86" y2="17.78" width="0.1524" layer="91"/>
-<wire x1="22.86" y1="17.78" x2="10.16" y2="17.78" width="0.1524" layer="91"/>
-<junction x="22.86" y="17.78"/>
-<label x="10.16" y="17.78" size="1.27" layer="95" rot="R180" xref="yes"/>
-<pinref part="S2" gate="G$1" pin="1"/>
-</segment>
-<segment>
 <pinref part="U1" gate="G$1" pin="PA06(AIN6/SER0:2/TC1:0)"/>

Commit message: working on sample libary and IMU
Parts:
- removed JP2: FTDI Basic, SparkFun:ARDUINO_SERIAL_PROGRAMPTH
Connections:
- removed net DTR: JP2.DTR
- removed net PROG: U1.PA06(AIN6/SER0:2/TC1:0)
- net GND: no longer JP2.CTS, JP2.GND
- net RXI: no longer JP2.TXO
- net TXO: no longer JP2.RXI
Changed lines of the file:
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@@
 <part name="R23" library="SparkFun-Resistors" deviceset="RESISTOR" device="0402" value="63"/>
 <part name="GND51" library="SparkFun-Aesthetics" deviceset="GND" device=""/>
-<part name="JP2" library="SparkFun" deviceset="ARDUINO_SERIAL_PROGRAM" device="PTH" value="FTDI Basic"/>
 <part name="R28" library="SparkFun-Passives" deviceset="RESISTOR" device="0402-RES" value="10k"/>
 <part name="SUPPLY15" library="SparkFun-Aesthetics" deviceset="3.3V" device=""/>
@@
 </instance>
 <instance part="GND51" gate="1" x="363.22" y="259.08" rot="R90"/>
-<instance part="JP2" gate="G$1" x="20.32" y="119.38"/>
 <instance part="R28" gate="G$1" x="401.32" y="200.66" rot="MR90"/>
 <instance part="SUPPLY15" gate="G$1" x="401.32" y="205.74"/>
@@
 </segment>
 <segment>
-<wire x1="25.4" y1="124.46" x2="27.94" y2="124.46" width="0.1524" layer="91"/>
-<pinref part="JP2" gate="G$1" pin="CTS"/>
-<label x="27.94" y="124.46" size="1.27" layer="95" xref="yes"/>
-</segment>
-<segment>
-<wire x1="25.4" y1="127" x2="27.94" y2="127" width="0.1524" layer="91"/>
-<pinref part="JP2" gate="G$1" pin="GND"/>
-<label x="27.94" y="127" size="1.27" layer="95" xref="yes"/>
-</segment>
-<segment>
 <pinref part="GND22" gate="1" pin="GND"/>
 <wire x1="147.32" y1="261.62" x2="144.78" y2="261.62" width="0.1524" layer="91"/>
@@
 <wire x1="241.3" y1="124.46" x2="243.84" y2="124.46" width="0.1524" layer="91"/>
 <label x="243.84" y="124.46" size="1.778" layer="95"/>
-</segment>
-</net>
-<net name="PROG" class="0">
-<segment>
-<pinref part="U1" gate="G$1" pin="PA06(AIN6/SER0:2/TC1:0)"/>
-<wire x1="172.72" y1="137.16" x2="170.18" y2="137.16" width="0.1524" layer="91"/>
-<label x="170.18" y="137.16" size="1.778" layer="95" rot="R180"/>
 </segment>
 </net>
@@
 <pinref part="U2" gate="G$1" pin="AD0/SDO"/>
 <wire x1="393.7" y1="187.96" x2="396.24" y2="187.96" width="0.1524" layer="91"/>
-<label x="396.24" y="187.96" size="1.778" layer="95"/>
+<label x="396.24" y="187.96" size="1.27" layer="95" xref="yes"/>
 </segment>
 <segment>
@@
 <pinref part="U2" gate="G$1" pin="SDA/SDI"/>
 <wire x1="393.7" y1="190.5" x2="396.24" y2="190.5" width="0.1524" layer="91"/>
-<label x="396.24" y="190.5" size="1.778" layer="95"/>
+<label x="396.24" y="190.5" size="1.27" layer="95" xref="yes"/>
 </segment>
 <segment>
 <pinref part="U3" gate="G$1" pin="SDA/SDI"/>
 <wire x1="360.68" y1="134.62" x2="358.14" y2="134.62" width="0.1524" layer="91"/>
-<label x="358.14" y="134.62" size="1.778" layer="95" rot="R180"/>
+<label x="358.14" y="134.62" size="1.27" layer="95" rot="R180" xref="yes"/>
 </segment>
 <segment>
@@
 <pinref part="U2" gate="G$1" pin="!CS"/>
 <wire x1="393.7" y1="195.58" x2="401.32" y2="195.58" width="0.1524" layer="91"/>
-<label x="408.94" y="195.58" size="1.778" layer="95"/>
+<label x="408.94" y="195.58" size="1.27" layer="95" xref="yes"/>
 <pinref part="R28" gate="G$1" pin="1"/>
 <wire x1="401.32" y1="195.58" x2="408.94" y2="195.58" width="0.1524" layer="91"/>
@@
 <pinref part="R3" gate="G$1" pin="1"/>
 <wire x1="388.62" y1="127" x2="403.86" y2="127" width="0.1524" layer="91"/>
-<wire x1="403.86" y1="127" x2="411.48" y2="127" width="0.1524" layer="91"/>
+<wire x1="403.86" y1="127" x2="408.94" y2="127" width="0.1524" layer="91"/>
 <junction x="403.86" y="127"/>
-<label x="411.48" y="127" size="1.778" layer="95" rot="R180"/>
+<label x="408.94" y="127" size="1.27" layer="95" xref="yes"/>
 </segment>
 <segment>
@@
 </segment>
 </net>
-<net name="DTR" class="0">
-<segment>
-<wire x1="25.4" y1="114.3" x2="27.94" y2="114.3" width="0.1524" layer="91"/>
-<pinref part="JP2" gate="G$1" pin="DTR"/>
-<label x="27.94" y="114.3" size="1.27" layer="95" xref="yes"/>
-</segment>
-</net>
 <net name="TXO" class="0">
-<segment>
-<wire x1="25.4" y1="116.84" x2="27.94" y2="116.84" width="0.1524" layer="91"/>
-<pinref part="JP2" gate="G$1" pin="RXI"/>
-<label x="27.94" y="116.84" size="1.27" layer="95" xref="yes"/>
-</segment>
 <segment>
 <pinref part="U1" gate="G$1" pin="PA08(I2C/AIN16/SER0:0+)"/>
@@
 </net>
 <net name="RXI" class="0">
-<segment>
-<wire x1="25.4" y1="119.38" x2="27.94" y2="119.38" width="0.1524" layer="91"/>
-<pinref part="JP2" gate="G$1" pin="TXO"/>
-<label x="27.94" y="119.38" size="1.27" layer="95" xref="yes"/>
-</segment>
 <segment>
 <pinref part="U1" gate="G$1" pin="PA09(I2C/AIN17/SER0:1+)"/>
@@
 <pinref part="U3" gate="G$1" pin="SCL/SCLK"/>
 <wire x1="360.68" y1="132.08" x2="358.14" y2="132.08" width="0.1524" layer="91"/>
-<label x="358.14" y="132.08" size="1.778" layer="95" rot="R180"/>
+<label x="358.14" y="132.08" size="1.27" layer="95" rot="R180" xref="yes"/>
 </segment>
 <segment>
 <pinref part="U2" gate="G$1" pin="SCL/SCLK"/>
 <wire x1="393.7" y1="193.04" x2="396.24" y2="193.04" width="0.1524" layer="91"/>
-<label x="396.24" y="193.04" size="1.778" layer="95"/>
-</segment>
-<segment>
+<label x="396.24" y="193.04" size="1.27" layer="95" xref="yes"/>
+</segment>
+<segment>

Commit message: changes to eagle stuff
Parts:
- R10, R12, R16, R22: value 27K -> (none)
- R11, R15, R21, R9: value 100K -> (none)
- R14, R17, R6, R7: value 100 -> (none)
- R20, R4, R5, R8: value 3.3k -> (none)
- R23: value 63 -> (none)
Changed lines of the file:
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@@
 <?xml version="1.0" encoding="utf-8"?>
 <!DOCTYPE eagle SYSTEM "eagle.dtd">
-<eagle version="8.3.2">
+<eagle version="8.4.0">
 <drawing>
 <settings>
@@
 <part name="GND19" library="SparkFun-Aesthetics" deviceset="GND" device=""/>
 <part name="GND20" library="SparkFun-Aesthetics" deviceset="GND" device=""/>
-<part name="R5" library="SparkFun-Resistors" deviceset="RESISTOR" device="0402" value="3.3k"/>
-<part name="R6" library="SparkFun-Resistors" deviceset="RESISTOR" device="0402" value="100"/>
-<part name="R9" library="SparkFun-Resistors" deviceset="RESISTOR" device="0402" value="100K"/>
-<part name="R10" library="SparkFun-Resistors" deviceset="RESISTOR" device="0402" value="27K"/>
-<part name="R7" library="SparkFun-Resistors" deviceset="RESISTOR" device="0402" value="100"/>
-<part name="R8" library="SparkFun-Resistors" deviceset="RESISTOR" device="0402" value="3.3k"/>
-<part name="R11" library="SparkFun-Resistors" deviceset="RESISTOR" device="0402" value="100K"/>
-<part name="R12" library="SparkFun-Resistors" deviceset="RESISTOR" device="0402" value="27K"/>
+<part name="R5" library="SparkFun-Resistors" library_urn="urn:adsk.eagle:library:532" deviceset="RESISTOR" device="0402" package3d_urn="urn:adsk.eagle:package:39657/1" value=" "/>
+<part name="R6" library="SparkFun-Resistors" library_urn="urn:adsk.eagle:library:532" deviceset="RESISTOR" device="0402" package3d_urn="urn:adsk.eagle:package:39657/1" value=" "/>
+<part name="R9" library="SparkFun-Resistors" library_urn="urn:adsk.eagle:library:532" deviceset="RESISTOR" device="0402" package3d_urn="urn:adsk.eagle:package:39657/1" value=" "/>
+<part name="R10" library="SparkFun-Resistors" library_urn="urn:adsk.eagle:library:532" deviceset="RESISTOR" device="0402" package3d_urn="urn:adsk.eagle:package:39657/1" value=" "/>
+<part name="R7" library="SparkFun-Resistors" library_urn="urn:adsk.eagle:library:532" deviceset="RESISTOR" device="0402" package3d_urn="urn:adsk.eagle:package:39657/1" value=" "/>
+<part name="R8" library="SparkFun-Resistors" library_urn="urn:adsk.eagle:library:532" deviceset="RESISTOR" device="0402" package3d_urn="urn:adsk.eagle:package:39657/1" value=" "/>
+<part name="R11" library="SparkFun-Resistors" library_urn="urn:adsk.eagle:library:532" deviceset="RESISTOR" device="0402" package3d_urn="urn:adsk.eagle:package:39657/1" value=" "/>
+<part name="R12" library="SparkFun-Resistors" library_urn="urn:adsk.eagle:library:532" deviceset="RESISTOR" device="0402" package3d_urn="urn:adsk.eagle:package:39657/1" value=" "/>
 <part name="SG1" library="SparkFun-Electromechanical" deviceset="BUZZER" device="SMD2"/>
 <part name="GND47" library="SparkFun-Aesthetics" deviceset="GND" device=""/>
@@
 <part name="SUPPLY1" library="SparkFun-Aesthetics" deviceset="3.3V" device=""/>
 <part name="GND1" library="SparkFun-Aesthetics" deviceset="GND" device=""/>
-<part name="C1" library="SparkFun-Capacitors" deviceset="CAP" device="0603-CAP" value="2.2uF"/>
-<part name="C2" library="SparkFun-Capacitors" deviceset="CAP" device="0603-CAP" value="2.2uF"/>
+<part name="C1" library="SparkFun-Capacitors" library_urn="urn:adsk.eagle:library:510" deviceset="CAP" device="0603-CAP" value="2.2uF"/>
+<part name="C2" library="SparkFun-Capacitors" library_urn="urn:adsk.eagle:library:510" deviceset="CAP" device="0603-CAP" value="2.2uF"/>
 <part name="U2" library="Testing" deviceset="MPU-9250" device=""/>
 <part name="GND2" library="SparkFun-Aesthetics" deviceset="GND" device=""/>
@@
 <part name="GND27" library="SparkFun-Aesthetics" deviceset="GND" device=""/>
 <part name="GND28" library="SparkFun-Aesthetics" deviceset="GND" device=""/>
-<part name="R4" library="SparkFun-Resistors" deviceset="RESISTOR" device="0402" value="3.3k"/>
-<part name="R14" library="SparkFun-Resistors" deviceset="RESISTOR" device="0402" value="100"/>
-<part name="R15" library="SparkFun-Resistors" deviceset="RESISTOR" device="0402" value="100K"/>
-<part name="R16" library="SparkFun-Resistors" deviceset="RESISTOR" device="0402" value="27K"/>
-<part name="R17" library="SparkFun-Resistors" deviceset="RESISTOR" device="0402" value="100"/>
-<part name="R20" library="SparkFun-Resistors" deviceset="RESISTOR" device="0402" value="3.3k"/>
-<part name="R21" library="SparkFun-Resistors" deviceset="RESISTOR" device="0402" value="100K"/>
-<part name="R22" library="SparkFun-Resistors" deviceset="RESISTOR" device="0402" value="27K"/>
+<part name="R4" library="SparkFun-Resistors" library_urn="urn:adsk.eagle:library:532" deviceset="RESISTOR" device="0402" package3d_urn="urn:adsk.eagle:package:39657/1" value=" "/>
+<part name="R14" library="SparkFun-Resistors" library_urn="urn:adsk.eagle:library:532" deviceset="RESISTOR" device="0402" package3d_urn="urn:adsk.eagle:package:39657/1" value=" "/>
+<part name="R15" library="SparkFun-Resistors" library_urn="urn:adsk.eagle:library:532" deviceset="RESISTOR" device="0402" package3d_urn="urn:adsk.eagle:package:39657/1" value=" "/>
+<part name="R16" library="SparkFun-Resistors" library_urn="urn:adsk.eagle:library:532" deviceset="RESISTOR" device="0402" package3d_urn="urn:adsk.eagle:package:39657/1" value=" "/>
+<part name="R17" library="SparkFun-Resistors" library_urn="urn:adsk.eagle:library:532" deviceset="RESISTOR" device="0402" package3d_urn="urn:adsk.eagle:package:39657/1" value=" "/>
+<part name="R20" library="SparkFun-Resistors" library_urn="urn:adsk.eagle:library:532" deviceset="RESISTOR" device="0402" package3d_urn="urn:adsk.eagle:package:39657/1" value=" "/>
+<part name="R21" library="SparkFun-Resistors" library_urn="urn:adsk.eagle:library:532" deviceset="RESISTOR" device="0402" package3d_urn="urn:adsk.eagle:package:39657/1" value=" "/>
+<part name="R22" library="SparkFun-Resistors" library_urn="urn:adsk.eagle:library:532" deviceset="RESISTOR" device="0402" package3d_urn="urn:adsk.eagle:package:39657/1" value=" "/>
 <part name="X1" library="con-molex" library_urn="urn:adsk.eagle:library:165" deviceset="22-23-2041" device=""/>
 <part name="X2" library="con-molex" library_urn="urn:adsk.eagle:library:165" deviceset="22-23-2041" device=""/>
 <part name="D2" library="SparkFun-LED" deviceset="LED-GREEN" device="1206" value="GREEN"/>
-<part name="R23" library="SparkFun-Resistors" deviceset="RESISTOR" device="0402" value="63"/>
+<part name="R23" library="SparkFun-Resistors" library_urn="urn:adsk.eagle:library:532" deviceset="RESISTOR" device="0402" package3d_urn="urn:adsk.eagle:package:39657/1" value=" "/>
 <part name="GND51" library="SparkFun-Aesthetics" deviceset="GND" device=""/>
 <part name="R28" library="SparkFun-Passives" deviceset="RESISTOR" device="0402-RES" value="10k"/>
@@
 with this version.
 </note>
+<note version="8.3" severity="warning">
+Since Version 8.3, EAGLE supports URNs for individual library
+assets (packages, symbols, and devices). The URNs of those assets
+will not be understood (or retained) with this version.
+</note>
+<note version="8.3" severity="warning">
+Since Version 8.3, EAGLE supports the association of 3D packages
+with devices in libraries, schematics, and board files. Those 3D
+packages will not be understood (or retained) with this version.
+</note>
 </compatibility>
