File: DasAltimeter V0.1/DasAltimeter V0.1/DasAltimeter V0.1.sch (EAGLE design)
At the start: 57 parts, among them IC1 BMI055, U1 ATSAMD21G-A, U2 3.3V/150mA, U3 MS5803-14BA, U4 ADXL193, X1 22-23-2041, X2 22-23-2041, Y1 32.768kHz

Commit message: V0.1 board
Parts:
- removed C6: 0.1uF, SparkFun-Capacitors:0.1UF-0402-16V-10%
Connections:
- removed net N$11: U1.PA24(SER3:2+)
- removed net N$14: U1.PA25(SER3:3+)
- removed net RESET: R1.1, U1.!RESET!
- new net RX: JP1.SWO/TDO, U1.PA23(I2C/SER3:0+)
- new net TX: JP1.NC/TDI, U1.PA22(I2C/SER3:0+)
- net !RESET: now also R1.1, U1.!RESET!
- net 3.3V: no longer C6.1
- net BUZZER: now also U1.PA21(SER5:3+); no longer U1.PA22(I2C/SER3:0+)
- net CS_ACCEL: now also U1.PB10(SER4:2+); no longer U1.PA10(AIN18/SER0:2+)
- net CS_BARO: now also U1.PA15(XOUT/SER2:3+); no longer U1.PA14(XIN/SER2:2+)
- net CS_GYRO: now also U1.PA10(AIN18/SER0:2+); no longer U1.PB10(SER4:2+)
- net FIRE_A: now also U1.PB23(SER5:3+)
- net FIRE_B: now also U1.PB22(SER5:2+)
- net FIRE_C: now also U1.PA25(SER3:3+)
- net FIRE_D: now also U1.PA24(SER3:2+)
- net GND: now also U1.GND@18, U1.GND@35, U1.GND@42, U1.GNDANA; no longer C6.2
- net LED: now also U1.PA20(SER5:2+)
- net SENSE_A: now also U1.PB03(AIN11/SER5:1); no longer U1.PB02(AIN10/SER5:0)
- net SENSE_B: now also U1.PB02(AIN10/SER5:0); no longer U1.PB03(AIN11/SER5:1)
- net SPI2_MISO: now also U1.PA13(I2C/SER2:1+); no longer U1.PA15(XOUT/SER2:3+)
- net SPI2_SCK: now also U1.PA14(XIN/SER2:2+); no longer U1.PA13(I2C/SER2:1+)

Commit message: DasAltimeter V0.1 sent to fab
Connections:
- removed net N$9: U1.PA28
Changed lines of the file:
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@@
-</segment>
-</net>
-<net name="N$9" class="0">
-<segment>
-<pinref part="U1" gate="G$1" pin="PA28"/>
-<wire x1="231.14" y1="111.76" x2="233.68" y2="111.76" width="0.1524" layer="91"/>
 </segment>
 </net>
@@
 </sheet>
 </sheets>
+<errors>
+</errors>
 </schematic>
 </drawing>

Commit message: setting up software
Connections:
- net CS_BARO: now also U1.PA14(XIN/SER2:2+); no longer U1.PA15(XOUT/SER2:3+)
- net SPI2_SCK: now also U1.PA15(XOUT/SER2:3+); no longer U1.PA14(XIN/SER2:2+)
Changed lines of the file:
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@@
 </segment>
 <segment>
-<pinref part="U1" gate="G$1" pin="PA14(XIN/SER2:2+)"/>
-<wire x1="231.14" y1="144.78" x2="233.68" y2="144.78" width="0.1524" layer="91"/>
-<label x="233.68" y="144.78" size="1.27" layer="95" xref="yes"/>
+<pinref part="U1" gate="G$1" pin="PA15(XOUT/SER2:3+)"/>
+<wire x1="231.14" y1="142.24" x2="233.68" y2="142.24" width="0.1524" layer="91"/>
+<label x="233.68" y="142.24" size="1.27" layer="95" xref="yes"/>
 </segment>
 </net>
@@
 </segment>
 <segment>
-<pinref part="U1" gate="G$1" pin="PA15(XOUT/SER2:3+)"/>
-<wire x1="231.14" y1="142.24" x2="233.68" y2="142.24" width="0.1524" layer="91"/>
-<label x="233.68" y="142.24" size="1.27" layer="95" xref="yes"/>
+<pinref part="U1" gate="G$1" pin="PA14(XIN/SER2:2+)"/>
+<wire x1="231.14" y1="144.78" x2="233.68" y2="144.78" width="0.1524" layer="91"/>
+<label x="233.68" y="144.78" size="1.27" layer="95" xref="yes"/>
 </segment>
 </net>
