File: Track'em V0.1/Track'em V0.1/Track'em V0.1.brd (EAGLE design)
At the start: 47.2 x 17 mm, 34 parts, among them IC1 SAM-M8Q, J1 CORTEX_DEBUG_PTH, U2 3.3V/150mA

Commit message: track'em updates
Parts:
- moved R2 0.51 mm to (34.0, 2.79)
Routing:
- net USART_TX: track 0.00 -> 26.7 mm
- net USART_RX: track 0.00 -> 26.0 mm, vias 0 -> 1
- net SWDCLK: track 13.9 -> 38.4 mm
- net SWDIO: track 14.3 -> 35.6 mm, vias 1 -> 0
- net RST: track 17.1 -> 26.9 mm, vias 2 -> 1
- net 3.3V: track 39.7 -> 40.6 mm, vias 16 -> 17
- net GND: vias 46 -> 49
Other:
- board text added: "Track'em v0.1"

Commit message: boards sent to fab
Connections:
- net GND: now also U$1.P$1, U$1.P$2, U$1.P$3, U$1.P$4, U$1.P$5
Routing:
- net GND: track 13.4 -> 12.6 mm, vias 49 -> 45
Changed lines of the file:
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@@
 <layer number="37" name="tTest" color="7" fill="1" visible="no" active="yes"/>
 <layer number="38" name="bTest" color="7" fill="1" visible="no" active="yes"/>
-<layer number="39" name="tKeepout" color="4" fill="11" visible="yes" active="yes"/>
-<layer number="40" name="bKeepout" color="1" fill="11" visible="yes" active="yes"/>
-<layer number="41" name="tRestrict" color="4" fill="10" visible="yes" active="yes"/>
+<layer number="39" name="tKeepout" color="4" fill="11" visible="no" active="yes"/>
+<layer number="40" name="bKeepout" color="1" fill="11" visible="no" active="yes"/>
+<layer number="41" name="tRestrict" color="4" fill="10" visible="no" active="yes"/>
 <layer number="42" name="bRestrict" color="1" fill="10" visible="yes" active="yes"/>
 <layer number="43" name="vRestrict" color="2" fill="10" visible="yes" active="yes"/>
@@
 </class>
 </classes>
-<designrules name="oshpark-4layer-tented">
+<designrules name="oshpark-4layer-tented *">
 <description language="en">&lt;b&gt;OSH Park Design Rules&lt;/b&gt;
 &lt;p&gt;
@@
 <param name="mvStopFrame" value="1"/>
 <param name="mvCreamFrame" value="0"/>
-<param name="mlMinStopFrame" value="2.5mil"/>
-<param name="mlMaxStopFrame" value="2.5mil"/>
+<param name="mlMinStopFrame" value="1.5mil"/>
+<param name="mlMaxStopFrame" value="1.5mil"/>
 <param name="mlMinCreamFrame" value="0mil"/>
 <param name="mlMaxCreamFrame" value="0mil"/>
@@
 <wire x1="17.78" y1="5.888" x2="17.78" y2="4.627" width="0.4064" layer="1"/>
 <wire x1="17.78" y1="4.627" x2="17.835" y2="4.572" width="0.4064" layer="1"/>
-<via x="28.194" y="11.43" extent="1-16" drill="0.254"/>
-<via x="28.956" y="11.43" extent="1-16" drill="0.254"/>
-<via x="28.956" y="10.668" extent="1-16" drill="0.254"/>
-<via x="28.194" y="10.668" extent="1-16" drill="0.254"/>
 <via x="35.56" y="15.24" extent="1-16" drill="0.254"/>
 <via x="38.1" y="15.24" extent="1-16" drill="0.254"/>
@@
 <vertex x="0" y="0"/>
 <vertex x="47.244" y="0"/>
-<vertex x="47.244" y="18.288"/>
-<vertex x="0" y="18.288"/>
+<vertex x="47.244" y="17.018"/>
+<vertex x="0" y="17.018"/>
 </polygon>
 <polygon width="0.254" layer="2">
 <vertex x="0" y="0"/>
-<vertex x="0" y="19.558"/>
-<vertex x="47.498" y="19.558"/>
+<vertex x="0" y="17.018"/>
+<vertex x="47.498" y="17.018"/>
 <vertex x="47.498" y="0"/>
 </polygon>
@@
 <vertex x="0" y="0"/>
 <vertex x="47.498" y="0"/>
-<vertex x="47.498" y="22.352"/>
-<vertex x="0" y="22.352"/>
+<vertex x="47.498" y="17.018"/>
+<vertex x="0" y="17.018"/>
 </polygon>
 <contactref element="IC1" pad="10"/>
@@
 <contactref element="IC1" pad="1"/>
 <contactref element="IC1" pad="15"/>
-<wire x1="28.575" y1="11.049" x2="28.575" y2="10.668" width="0.254" layer="1"/>
-<wire x1="28.575" y1="10.668" x2="28.194" y2="10.668" width="0.254" layer="1"/>
 <via x="1.27" y="6.35" extent="1-16" drill="0.254"/>
 <via x="1.27" y="4.318" extent="1-16" drill="0.254"/>
@@
 <via x="43.434" y="13.462" extent="1-16" drill="0.35"/>
 <via x="45.72" y="13.462" extent="1-16" drill="0.35"/>
+<contactref element="U$1" pad="P$1"/>
+<contactref element="U$1" pad="P$2"/>
+<contactref element="U$1" pad="P$3"/>
+<contactref element="U$1" pad="P$4"/>
+<contactref element="U$1" pad="P$5"/>
 </signal>
 <signal name="3.3V">
@@
 <polygon width="0.254" layer="15">
 <vertex x="0" y="0"/>
-<vertex x="0" y="20.828"/>
-<vertex x="47.498" y="20.828"/>
+<vertex x="0" y="17.018"/>
+<vertex x="47.498" y="17.018"/>
 <vertex x="47.498" y="0"/>
 </polygon>
@@
 </signal>
 </signals>
+<errors>
+</errors>
 </board>
 </drawing>

Commit message: this Track'em sent to fab
Parts:
- added C16: 10uF, SparkFun-Capacitors:0603-POL
- C10, C7: value 0.1uF -> 10nF
- C11, C12, C9: value 0.1uF -> 220pF
- C13: value 0.1uF -> 12pF
- C14: value 0.1uF -> 15pF
- C5, C6: value 0.1uF -> 100nF
- R1: value 10k -> 56k
- Y1: value (none) -> 26MHz
- moved C7 0.25 mm to (29.1, 6.96)
Connections:
- net 3.3V: now also C16.A, R3.1
- net GND: now also C16.K; no longer R3.1
Routing:
- net GND: track 12.6 -> 17.0 mm
- net 3.3V: track 40.6 -> 43.7 mm, vias 17 -> 18
- net USART_TX: track 26.7 -> 27.7 mm
- net USART_RX: track 26.0 -> 27.1 mm

Commit message: tracking message parsed from GPS
Connections:
- net USART_RX: now also U$2.9; no longer U$2.10
- net USART_TX: now also U$2.10; no longer U$2.9
Routing:
- net USART_TX: track 27.7 -> 23.6 mm
- net USART_RX: track 27.1 -> 23.7 mm
Changed lines of the file:
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@@
 <signal name="USART_RX">
 <contactref element="J1" pad="6"/>
-<contactref element="U$2" pad="10"/>
 <wire x1="37.973" y1="3.048" x2="37.973" y2="3.683" width="0.254" layer="16"/>
 <wire x1="37.973" y1="3.683" x2="37.084" y2="4.572" width="0.254" layer="16"/>
 <wire x1="37.084" y1="4.572" x2="34.036" y2="4.572" width="0.254" layer="16"/>
 <wire x1="32.512" y1="3.048" x2="34.036" y2="4.572" width="0.254" layer="16"/>
-<wire x1="16.51" y1="5.888" x2="16.51" y2="2.54" width="0.254" layer="1"/>
 <wire x1="16.51" y1="2.54" x2="17.018" y2="2.032" width="0.254" layer="1"/>
 <wire x1="24.638" y1="2.032" x2="25.654" y2="3.048" width="0.254" layer="1"/>
@@
 <wire x1="17.018" y1="2.032" x2="24.638" y2="2.032" width="0.254" layer="1"/>
 <wire x1="25.654" y1="3.048" x2="32.512" y2="3.048" width="0.254" layer="16"/>
+<contactref element="U$2" pad="9"/>
+<wire x1="16.51" y1="2.54" x2="15.24" y2="5.888" width="0" layer="19" extent="1-1"/>
 </signal>
 <signal name="USART_TX">
 <contactref element="J1" pad="8"/>
-<contactref element="U$2" pad="9"/>
 <wire x1="36.703" y1="3.048" x2="36.703" y2="3.683" width="0.254" layer="16"/>
 <wire x1="36.322" y1="4.064" x2="34.544" y2="4.064" width="0.254" layer="16"/>
 <wire x1="32.766" y1="2.286" x2="34.544" y2="4.064" width="0.254" layer="16"/>
 <wire x1="36.703" y1="3.683" x2="36.322" y2="4.064" width="0.254" layer="16"/>
-<wire x1="15.24" y1="5.888" x2="15.24" y2="1.778" width="0.254" layer="1"/>
 <wire x1="15.24" y1="1.778" x2="15.748" y2="1.27" width="0.254" layer="1"/>
 <wire x1="25.146" y1="1.27" x2="26.162" y2="2.286" width="0.254" layer="1"/>
@@
 <wire x1="15.748" y1="1.27" x2="25.146" y2="1.27" width="0.254" layer="1"/>
 <wire x1="26.162" y1="2.286" x2="32.766" y2="2.286" width="0.254" layer="16"/>
+<contactref element="U$2" pad="10"/>
+<wire x1="15.24" y1="1.778" x2="16.51" y2="5.888" width="0" layer="19" extent="1-1"/>
 </signal>
 <signal name="RAW">
