File: Track'em V0.2/Track'em V0.2/Track'em V0.2.sch (EAGLE design)
At the start: 36 parts, among them IC1 SAM-M8Q, J1 CORTEX_DEBUG_PTH, U2 3.3V/150mA, Y1 26MHz

Commit message: fix GPS for trackem v0.2
Connections:
- net 3.3V: now also IC1.VCC_IO, IC1.V_BCKP
Changed lines of the file:
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@@
 <part name="C17" library="SparkFun-Capacitors" deviceset="0.1UF" device="-0402-16V-10%" value="0.1uF"/>
 <part name="GND3" library="SparkFun-Aesthetics" deviceset="GND" device=""/>
+<part name="SUPPLY11" library="SparkFun-Aesthetics" deviceset="3.3V" device=""/>
 </parts>
 <sheets>
@@
 <instance part="C17" gate="G$1" x="208.28" y="154.94"/>
 <instance part="GND3" gate="1" x="208.28" y="149.86"/>
+<instance part="SUPPLY11" gate="G$1" x="177.8" y="71.12"/>
 </instances>
 <busses>
@@
 <pinref part="SUPPLY8" gate="G$1" pin="3.3V"/>
 </segment>
+<segment>
+<pinref part="IC1" gate="G$1" pin="V_BCKP"/>
+<pinref part="SUPPLY11" gate="G$1" pin="3.3V"/>
+<wire x1="182.88" y1="63.5" x2="177.8" y2="63.5" width="0.1524" layer="91"/>
+<wire x1="177.8" y1="63.5" x2="177.8" y2="68.58" width="0.1524" layer="91"/>
+<pinref part="IC1" gate="G$1" pin="VCC_IO"/>
+<wire x1="177.8" y1="68.58" x2="177.8" y2="71.12" width="0.1524" layer="91"/>
+<wire x1="182.88" y1="68.58" x2="177.8" y2="68.58" width="0.1524" layer="91"/>
+<junction x="177.8" y="68.58"/>
+</segment>
 </net>

Commit message: tracking message parsed from GPS
Parts:
- removed C3, C4: 1000pF, SparkFun-Capacitors:2.2UF-0603-10V-20%
- removed L1: 6.8nH, SparkFun-Passives:INDUCTOR0603
- added C18, C19: 1000pF, SparkFun-Capacitors:0.1UF-0402-16V-10%
- added L2: 6.8NH, SparkFun-Coils:INDUCTOR-0402-3.9NH
Connections:
- net N$1: now also L2.2; no longer L1.2
- net N$13: now also C19.2; no longer C4.2
- net N$2: now also C18.2, L2.1; no longer C3.2, L1.1
- net N$3: now also C19.1; no longer C4.1
- net UBAL: now also C18.1; no longer C3.1
- net USART_RX: now also U$2.PA24(USB_D-/SER1:2); no longer U$2.PA25(USB_D+/SER1:3)
- net USART_TX: now also U$2.PA25(USB_D+/SER1:3); no longer U$2.PA24(USB_D-/SER1:2)
Changed lines of the file:
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@@
 <part name="GND44" library="SparkFun-Aesthetics" deviceset="GND" device=""/>
 <part name="U$4" library="SaL-lib1" deviceset="AN26018A" device=""/>
-<part name="C3" library="SparkFun-Capacitors" deviceset="2.2UF" device="-0603-10V-20%" value="1000pF"/>
-<part name="L1" library="SparkFun-Passives" deviceset="INDUCTOR" device="0603" value="6.8nH"/>
-<part name="C4" library="SparkFun-Capacitors" deviceset="2.2UF" device="-0603-10V-20%" value="1000pF"/>
 <part name="H1" library="SparkFun-Hardware" deviceset="STAND-OFF" device="TIGHT"/>
 <part name="H2" library="SparkFun-Hardware" deviceset="STAND-OFF" device="TIGHT"/>
@@
 <part name="GND3" library="SparkFun-Aesthetics" deviceset="GND" device=""/>
 <part name="SUPPLY11" library="SparkFun-Aesthetics" deviceset="3.3V" device=""/>
+<part name="C18" library="SparkFun-Capacitors" deviceset="0.1UF" device="-0402-16V-10%" value="1000pF"/>
+<part name="C19" library="SparkFun-Capacitors" deviceset="0.1UF" device="-0402-16V-10%" value="1000pF"/>
+<part name="L2" library="SparkFun-Coils" library_urn="urn:adsk.eagle:library:512" deviceset="INDUCTOR" device="-0402-3.9NH" package3d_urn="urn:adsk.eagle:package:37575/1" value="6.8NH"/>
 </parts>
 <sheets>
@@
 <instance part="GND44" gate="1" x="243.84" y="172.72"/>
 <instance part="U$4" gate="G$1" x="193.04" y="165.1"/>
-<instance part="C3" gate="G$1" x="160.02" y="170.18" rot="R90"/>
-<instance part="L1" gate="G$1" x="170.18" y="170.18" rot="R90"/>
-<instance part="C4" gate="G$1" x="215.9" y="170.18" rot="R90"/>
 <instance part="H1" gate="G$1" x="88.9" y="25.4"/>
 <instance part="H2" gate="G$1" x="91.44" y="25.4"/>
@@
 <instance part="GND3" gate="1" x="208.28" y="149.86"/>
 <instance part="SUPPLY11" gate="G$1" x="177.8" y="71.12"/>
+<instance part="C18" gate="G$1" x="160.02" y="170.18" rot="R90"/>
+<instance part="C19" gate="G$1" x="215.9" y="170.18" rot="R90"/>
+<instance part="L2" gate="G$1" x="172.72" y="170.18" rot="R90"/>
 </instances>
 <busses>
@@
 <wire x1="233.68" y1="170.18" x2="218.44" y2="170.18" width="0.1524" layer="91"/>
 <pinref part="J$1" gate="1" pin="SIGNAL"/>
-<pinref part="C4" gate="G$1" pin="2"/>
+<pinref part="C19" gate="G$1" pin="2"/>
 </segment>
 </net>
@@
 <segment>
 <pinref part="U$4" gate="G$1" pin="IN"/>
-<pinref part="L1" gate="G$1" pin="2"/>
-<wire x1="175.26" y1="170.18" x2="180.34" y2="170.18" width="0.1524" layer="91"/>
+<wire x1="177.8" y1="170.18" x2="180.34" y2="170.18" width="0.1524" layer="91"/>
+<pinref part="L2" gate="G$1" pin="2"/>
 </segment>
 </net>
 <net name="N$2" class="0">
 <segment>
-<pinref part="L1" gate="G$1" pin="1"/>
-<pinref part="C3" gate="G$1" pin="2"/>
 <wire x1="162.56" y1="170.18" x2="167.64" y2="170.18" width="0.1524" layer="91"/>
+<pinref part="L2" gate="G$1" pin="1"/>
+<pinref part="C18" gate="G$1" pin="2"/>
 </segment>
 </net>
@@
 <segment>
 <pinref part="U$4" gate="G$1" pin="OUT"/>
-<pinref part="C4" gate="G$1" pin="1"/>
 <wire x1="210.82" y1="170.18" x2="205.74" y2="170.18" width="0.1524" layer="91"/>
+<pinref part="C19" gate="G$1" pin="1"/>
 </segment>
 </net>
 <net name="UBAL" class="0">
 <segment>
-<pinref part="C3" gate="G$1" pin="1"/>
 <wire x1="154.94" y1="170.18" x2="147.32" y2="170.18" width="0.1524" layer="91"/>
 <label x="147.32" y="170.18" size="1.778" layer="95" rot="R180"/>
+<pinref part="C18" gate="G$1" pin="1"/>
 </segment>
 <segment>
@@
 </segment>
 <segment>
+<pinref part="U$2" gate="G$1" pin="PA24(USB_D-/SER1:2)"/>
+<wire x1="93.98" y1="91.44" x2="91.44" y2="91.44" width="0.1524" layer="91"/>
+<label x="91.44" y="91.44" size="1.27" layer="95" rot="R180" xref="yes"/>
+</segment>
+</net>
+<net name="USART_TX" class="0">
+<segment>
+<pinref part="J1" gate="G$1" pin="NC/TDI"/>
+<wire x1="218.44" y1="134.62" x2="220.98" y2="134.62" width="0.1524" layer="91"/>
+<label x="220.98" y="134.62" size="1.27" layer="95" xref="yes"/>
+</segment>
+<segment>
 <pinref part="U$2" gate="G$1" pin="PA25(USB_D+/SER1:3)"/>
 <wire x1="93.98" y1="93.98" x2="91.44" y2="93.98" width="0.1524" layer="91"/>
@@
 </segment>
 </net>
-<net name="USART_TX" class="0">
-<segment>
-<pinref part="J1" gate="G$1" pin="NC/TDI"/>
-<wire x1="218.44" y1="134.62" x2="220.98" y2="134.62" width="0.1524" layer="91"/>
-<label x="220.98" y="134.62" size="1.27" layer="95" xref="yes"/>
-</segment>
-<segment>
-<pinref part="U$2" gate="G$1" pin="PA24(USB_D-/SER1:2)"/>
-<wire x1="93.98" y1="91.44" x2="91.44" y2="91.44" width="0.1524" layer="91"/>
-<label x="91.44" y="91.44" size="1.27" layer="95" rot="R180" xref="yes"/>
-</segment>
-</net>

Commit message: setting up trackem v0.2
Parts:
- removed C18: 1000pF, SparkFun-Capacitors:0.1UF-0402-16V-10%
- removed U$3: 0433BM15A0001, SaL-lib1:0433BM15A0001
- removed U$4: AN26018A, SaL-lib1:AN26018A
- added C20, C21: 1000pF, SparkFun-Capacitors:0.1UF-0402-16V-10%
- added C3: 3.9pF, SparkFun-Capacitors:0.1UF-0402-16V-10%
- added C4: 8.2pF, SparkFun-Capacitors:0.1UF-0402-16V-10%
- added L1, L3: 27NH, SparkFun-Coils:INDUCTOR-0402-3.9NH
- added L4: 6.8NH, SparkFun-Coils:INDUCTOR-0402-3.9NH
- C17: value 0.1uF -> 220pF
Connections:
- removed net N$13: C19.2, J$1.SIGNAL
- removed net UBAL: C18.1, U$3.UNBAL
- new net ANT: C21.2, J$1.SIGNAL
- new net N$5: C20.1, C21.1, L2.2
- net 3.3V: no longer C17.1, U$4.VCC
- net CNT: no longer U$4.CNT
- net GND: now also C3.2; no longer U$3.GND, U$3.GND1, U$3.GND2, U$4.GND
- net N$1: now also C17.1, L1.1; no longer L2.2, U$4.IN
- net N$2: now also C4.1, L3.2, L4.1; no longer C18.2, L2.1
- net N$3: now also L2.1, L4.2; no longer U$4.OUT
- net RF_N: now also C3.1, L3.1; no longer U$3.BAL
- net RF_P: now also C4.2, L1.2; no longer U$3.BAL1
Other:
- moved on the sheet: C17, C19, L2
