File: Girlfriend Tracker V0.2/Girlfriend Tracker V0.2.brd (EAGLE design)
At the start: 53.1 x 20.8 mm, 64 parts, among them IC1 SAM-M8Q, IC2 FT234XD, U1 3.6V/200mA - TLV70036DDCR, U3 ATSAMD21G-A, U4 3.6V/200mA - TLV70036DDCR, X1 SMA-142-0701-851/861, Y1 26MHz

Commit message: tracker work
Parts:
- removed TP1, TP2, TP3, TP4: TPSQTP06R, testpad:TP06R
- added JP1: CORTEX_DEBUG_PTH, SparkFun-Connectors:2X5-PTH-1.27MM
- moved C32 0.76 mm to (10.4, 9.65)
- moved R4 0.76 mm to (22.9, 18.0)
- moved U3 0.76 mm to (19.6, 11.7)
- moved C27 0.72 mm to (13.0, 12.2)
- moved C33 0.51 mm to (19.1, 5.84)
- moved IC2 0.51 mm to (24.4, 4.83)
- moved R8 0.51 mm to (25.7, 2.03)
- moved R9 0.51 mm to (23.1, 2.03)
- moved C6 0.51 mm to (27.2, 10.4)
- moved C36 0.25 mm to (21.1, 2.79)
- moved C37 0.25 mm to (27.7, 2.79)
Connections:
- removed net AMP_EM: U1.3, U3.38
- removed net VDD: IC2.2, IC2.3, IC2.9
- new net AMP_EN: U1.3, U3.33
- net !RESET: now also JP1.10; no longer TP3.TP
- net 3.3V: now also IC2.2, IC2.3, IC2.9, JP1.1
- net GND: now also JP1.3, JP1.5; no longer TP4.TP
- net RX: now also JP1.6, U3.38; no longer U3.34
- net SER5_RX: no longer U3.48
- net SER5_TX: no longer U3.47
- net SWCLK: now also JP1.4; no longer TP1.TP
- net SWDIO: now also JP1.2; no longer TP2.TP
- net TX: now also JP1.8, U3.37; no longer U3.33
Routing:
- net V_BATT: track 9.10 -> 45.1 mm, vias 0 -> 2
- net 3.3V: track 32.9 -> 53.2 mm, vias 7 -> 15
- net AMP_EN: track 0.00 -> 19.0 mm, vias 0 -> 2
- net GND: track 2.90 -> 15.5 mm, vias 0 -> 13
- net !RESET: track 0.00 -> 12.1 mm, vias 0 -> 1
- net SER0_MISO: track 0.00 -> 9.63 mm
- net CS_MEM: track 1.90 -> 10.9 mm
- net SER0_SCK: track 0.00 -> 8.31 mm
- net SER0_MOSI: track 0.00 -> 7.73 mm
- net SWCLK: track 4.33 -> 11.1 mm, vias 0 -> 1
- net RX: track 0.00 -> 5.71 mm
- net TX: track 0.00 -> 4.37 mm
- net SWDIO: track 6.12 -> 10.3 mm, vias 0 -> 1
- net N$29: track 0.00 -> 2.15 mm, vias 0 -> 1
- net N$2: track 23.2 -> 24.2 mm
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
Commit message: square mock up
Connections:
- removed net SER5_RX: IC1.13
- removed net SER5_TX: IC1.14
- new net GPS_RX: IC1.13, U3.2
- new net GPS_TX: IC1.14, U3.1
- net LED: now also U3.8
Routing:
- net LED: track 0.00 -> 12.4 mm, vias 0 -> 1
- net GND: track 15.5 -> 27.4 mm, vias 13 -> 47
- net GPS_RX: track 0.00 -> 5.61 mm, vias 0 -> 1
- net GPS_TX: track 0.00 -> 5.03 mm, vias 0 -> 1
- net 3.3V: track 53.2 -> 58.0 mm, vias 15 -> 16
- added copper zone on layer 15, net 3.3V
- added copper zone on layer 1, net GND
- added copper zone on layer 16, net GND
- added copper zone on layer 2, net GND

Commit message: test flight three
Parts:
- C10, C22, C7: value 0.1uF -> 10nF
- C11, C12, C9: value 0.1uF -> 220pF
- C17, C21: value 0.1uF -> 220pf
- C19: value 0.1uF -> 8.2pF
- C20: value 0.1uF -> 5.6pF
- C26: value 0.1uF -> 1uF
- C3, C4: value 0.1uF -> 3.9pF
- L2: value 6.8NH -> 27NH
- L4: value 6.8NH -> 22NH
Changed lines of the file:
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@@
 <?xml version="1.0" encoding="utf-8"?>
 <!DOCTYPE eagle SYSTEM "eagle.dtd">
-<eagle version="8.6.0">
+<eagle version="8.7.0">
 <drawing>
 <settings>
@@
 </autorouter>
 <elements>
-<element name="C10" library="SparkFun-Capacitors" package="0402" value="0.1uF" x="34.925" y="14.224" smashed="yes" rot="R270">
+<element name="C10" library="SparkFun-Capacitors" package="0402" value="10nF" x="34.925" y="14.224" smashed="yes" rot="R270">
 <attribute name="NAME" x="35.179" y="15.494" size="0.6096" layer="25" font="vector" ratio="20" align="bottom-center"/>
 <attribute name="PROD_ID" value="CAP-12416" x="34.925" y="14.224" size="1.778" layer="27" rot="R270" display="off"/>
 </element>
-<element name="C11" library="SparkFun-Capacitors" package="0402" value="0.1uF" x="33.401" y="14.224" smashed="yes" rot="R270">
+<element name="C11" library="SparkFun-Capacitors" package="0402" value="220pF" x="33.401" y="14.224" smashed="yes" rot="R270">
 <attribute name="NAME" x="33.274" y="15.494" size="0.6096" layer="25" font="vector" ratio="20" align="bottom-center"/>
 <attribute name="PROD_ID" value="CAP-12416" x="33.401" y="14.224" size="1.778" layer="27" rot="R270" display="off"/>
 </element>
-<element name="C12" library="SparkFun-Capacitors" package="0402" value="0.1uF" x="35.306" y="6.477" smashed="yes" rot="R180">
+<element name="C12" library="SparkFun-Capacitors" package="0402" value="220pF" x="35.306" y="6.477" smashed="yes" rot="R180">
 <attribute name="NAME" x="35.306" y="5.207" size="0.6096" layer="25" font="vector" ratio="20" align="bottom-center"/>
 <attribute name="PROD_ID" value="CAP-12416" x="35.306" y="6.477" size="1.778" layer="27" rot="R180" display="off"/>
@@
 <attribute name="PROD_ID" value="CAP-12416" x="33.782" y="4.699" size="1.778" layer="27" display="off"/>
 </element>
-<element name="C17" library="SparkFun-Capacitors" package="0402" value="0.1uF" x="36.83" y="7.874" smashed="yes">
+<element name="C17" library="SparkFun-Capacitors" package="0402" value="220pf" x="36.83" y="7.874" smashed="yes">
 <attribute name="NAME" x="38.227" y="6.985" size="0.6096" layer="25" font="vector" ratio="20" rot="R180" align="bottom-center"/>
 <attribute name="PROD_ID" value="CAP-12416" x="36.83" y="7.874" size="1.778" layer="27" display="off"/>
@@
 <attribute name="PROD_ID" value="CAP-12416" x="42.545" y="7.112" size="1.778" layer="27" display="off"/>
 </element>
-<element name="C19" library="SparkFun-Capacitors" package="0402" value="0.1uF" x="46.482" y="11.557" smashed="yes">
+<element name="C19" library="SparkFun-Capacitors" package="0402" value="8.2pF" x="46.482" y="11.557" smashed="yes">
 <attribute name="NAME" x="46.482" y="12.192" size="0.6096" layer="25" font="vector" ratio="20" align="bottom-center"/>
 <attribute name="PROD_ID" value="CAP-12416" x="46.482" y="11.557" size="1.778" layer="27" display="off"/>
 </element>
-<element name="C20" library="SparkFun-Capacitors" package="0402" value="0.1uF" x="43.942" y="15.621" smashed="yes" rot="R180">
+<element name="C20" library="SparkFun-Capacitors" package="0402" value="5.6pF" x="43.942" y="15.621" smashed="yes" rot="R180">
 <attribute name="NAME" x="43.942" y="16.256" size="0.6096" layer="25" font="vector" ratio="20" align="bottom-center"/>
 <attribute name="PROD_ID" value="CAP-12416" x="43.942" y="15.621" size="1.778" layer="27" rot="R180" display="off"/>
 </element>
-<element name="C21" library="SparkFun-Capacitors" package="0402" value="0.1uF" x="46.482" y="14.097" smashed="yes">
+<element name="C21" library="SparkFun-Capacitors" package="0402" value="220pf" x="46.482" y="14.097" smashed="yes">
 <attribute name="NAME" x="46.482" y="14.859" size="0.6096" layer="25" font="vector" ratio="20" align="bottom-center"/>
 <attribute name="PROD_ID" value="CAP-12416" x="46.482" y="14.097" size="1.778" layer="27" display="off"/>
 </element>
-<element name="C22" library="SparkFun-Capacitors" package="0402" value="0.1uF" x="39.37" y="13.462" smashed="yes" rot="R180">
+<element name="C22" library="SparkFun-Capacitors" package="0402" value="10nF" x="39.37" y="13.462" smashed="yes" rot="R180">
 <attribute name="NAME" x="39.37" y="12.192" size="0.6096" layer="25" font="vector" ratio="20" align="bottom-center"/>
 <attribute name="PROD_ID" value="CAP-12416" x="39.37" y="13.462" size="1.778" layer="27" rot="R180" display="off"/>
@@
 <attribute name="PROD_ID" value="CAP-12416" x="17.526" y="18.796" size="1.778" layer="27" rot="R180" display="off"/>
 </element>
-<element name="C26" library="SparkFun-Capacitors" package="0402" value="0.1uF" x="20.066" y="18.796" smashed="yes">
+<element name="C26" library="SparkFun-Capacitors" package="0402" value="1uF" x="20.066" y="18.796" smashed="yes">
 <attribute name="NAME" x="20.066" y="19.558" size="0.6096" layer="25" font="vector" ratio="20" align="bottom-center"/>
 <attribute name="PROD_ID" value="CAP-12416" x="20.066" y="18.796" size="1.778" layer="27" display="off"/>
@@
 <attribute name="PROD_ID" value="CAP-12416" x="12.954" y="12.192" size="1.778" layer="27" rot="R90" display="off"/>
 </element>
-<element name="C3" library="SparkFun-Capacitors" package="0402" value="0.1uF" x="34.798" y="11.43" smashed="yes" rot="R90">
+<element name="C3" library="SparkFun-Capacitors" package="0402" value="3.9pF" x="34.798" y="11.43" smashed="yes" rot="R90">
 <attribute name="NAME" x="35.941" y="11.811" size="0.6096" layer="25" font="vector" ratio="20" align="bottom-center"/>
 <attribute name="PROD_ID" value="CAP-12416" x="34.798" y="11.43" size="1.778" layer="27" rot="R90" display="off"/>
@@
 <attribute name="NAME" x="30.734" y="18.907" size="0.6096" layer="25" font="vector" ratio="20"/>
 </element>
-<element name="C4" library="SparkFun-Capacitors" package="0402" value="0.1uF" x="36.83" y="9.398" smashed="yes" rot="R180">
+<element name="C4" library="SparkFun-Capacitors" package="0402" value="3.9pF" x="36.83" y="9.398" smashed="yes" rot="R180">
 <attribute name="NAME" x="35.814" y="10.16" size="0.6096" layer="25" font="vector" ratio="20" rot="R180" align="bottom-center"/>
 <attribute name="PROD_ID" value="CAP-12416" x="36.83" y="9.398" size="1.778" layer="27" rot="R180" display="off"/>
@@
 <attribute name="PROD_ID" value="CAP-12416" x="27.178" y="10.414" size="1.778" layer="27" display="off"/>
 </element>
-<element name="C7" library="SparkFun-Capacitors" package="0402" value="0.1uF" x="32.258" y="6.731" smashed="yes" rot="R90">
+<element name="C7" library="SparkFun-Capacitors" package="0402" value="10nF" x="32.258" y="6.731" smashed="yes" rot="R90">
 <attribute name="NAME" x="31.496" y="6.731" size="0.6096" layer="25" font="vector" ratio="20" rot="R90" align="bottom-center"/>
 <attribute name="PROD_ID" value="CAP-12416" x="32.258" y="6.731" size="1.778" layer="27" rot="R90" display="off"/>
@@
 <attribute name="PROD_ID" value="CAP-12416" x="8.382" y="2.54" size="1.778" layer="27" rot="R90" display="off"/>
 </element>
-<element name="C9" library="SparkFun-Capacitors" package="0402" value="0.1uF" x="30.226" y="14.224" smashed="yes" rot="R270">
+<element name="C9" library="SparkFun-Capacitors" package="0402" value="220pF" x="30.226" y="14.224" smashed="yes" rot="R270">
 <attribute name="NAME" x="30.226" y="15.494" size="0.6096" layer="25" font="vector" ratio="20" align="bottom-center"/>
 <attribute name="PROD_ID" value="CAP-12416" x="30.226" y="14.224" size="1.778" layer="27" rot="R270" display="off"/>
@@
 <attribute name="PROD_ID" value="NDUC-13457" x="34.798" y="8.89" size="1.778" layer="27" rot="R90" display="off"/>
 </element>
-<element name="L2" library="SparkFun-Coils" library_urn="urn:adsk.eagle:library:512" package="0402" package3d_urn="urn:adsk.eagle:package:37575/1" value="6.8NH" x="44.45" y="13.589" smashed="yes" rot="R90">
+<element name="L2" library="SparkFun-Coils" library_urn="urn:adsk.eagle:library:512" package="0402" package3d_urn="urn:adsk.eagle:package:37575/1" value="27NH" x="44.45" y="13.589" smashed="yes" rot="R90">
 <attribute name="NAME" x="43.815" y="13.589" size="0.6096" layer="25" font="vector" ratio="20" rot="R90" align="bottom-center"/>
 <attribute name="PROD_ID" value="NDUC-13457" x="44.45" y="13.589" size="1.778" layer="27" rot="R90" display="off"/>
@@
 <attribute name="PROD_ID" value="NDUC-13457" x="36.83" y="10.795" size="1.778" layer="27" display="off"/>
 </element>
-<element name="L4" library="SparkFun-Coils" library_urn="urn:adsk.eagle:library:512" package="0402" package3d_urn="urn:adsk.eagle:package:37575/1" value="6.8NH" x="44.45" y="11.049" smashed="yes" rot="R90">
+<element name="L4" library="SparkFun-Coils" library_urn="urn:adsk.eagle:library:512" package="0402" package3d_urn="urn:adsk.eagle:package:37575/1" value="22NH" x="44.45" y="11.049" smashed="yes" rot="R90">
 <attribute name="NAME" x="44.45" y="9.779" size="0.6096" layer="25" font="vector" ratio="20" rot="R180" align="bottom-center"/>
 <attribute name="PROD_ID" value="NDUC-13457" x="44.45" y="11.049" size="1.778" layer="27" rot="R90" display="off"/>
