File: Girlfriend Tracker V0.2/Girlfriend Tracker V0.2.sch (EAGLE design)
At the start: 61 parts, among them IC1 SAM-M8Q, U1 3.6V/200mA - TLV70036DDCR, U2 3.6V/200mA - TLV70036DDCR, U3 ATSAMD21G-A, U4 3.6V/200mA - TLV70036DDCR, X1 SMA-142-0701-851/861, Y1 26MHz, Y2 32.768kHz

Commit message: girlfriend tracker board updates
Parts:
- removed C1, C2: 2.2uF, SparkFun-Capacitors:2.2UF-0603-10V-20%
- removed C15: 10uF, SparkFun:CAP_POL1206
- removed C16: 10uF, SparkFun-Capacitors:10UF-6.3V-20%(0603)(TANT)"
- removed C28, C29: 15pF, SparkFun-Capacitors:15PF-0402-50V-5%
- removed JP1: CORTEX_DEBUG_PTH, SparkFun-Connectors:CORTEX_DEBUG_PTH
- removed R3: 10k, SparkFun-Resistors:RESISTOR0402
- removed U2: 3.6V/200mA - TLV70036DDCR, SparkFun-IC-Power:V_REG_MIC52053.3V
- removed Y2: 32.768kHz, SparkFun-Clocks:CRYSTAL-32.768KHZSMD-3.2X1.5
- added C33: 0.1uF, SparkFun-Capacitors:0.1UF-0402-16V-10%
- added C34: 10uF, SparkFun:CAP_POL1206
- added C36, C37: 47pF, SparkFun-Capacitors:0.1UF-0402-16V-10%
- added IC2: FT234XD, ft234xd:FT234XD
- added JP2: USB-MICROB", SparkFun-Connectors:USB-MICROB"
- added R2: (no value), SparkFun-Resistors:RESISTOR0402
- added R8, R9: 27, SparkFun-Resistors:RESISTOR0402
- added TP1, TP2, TP3, TP4: TPSQTP06R, testpad:TPSQTP06R
- C10, C7: value 10nF -> 0.1uF
- C11, C12, C17, C9: value 220pF -> 0.1uF
- C13, C14: value 15pF -> 0.1uF
- C18, C22: value 0.01uF -> 0.1uF
- C19, C20, C21: value 1000pF -> 0.1uF
- C24: value 0.1uF -> 2.2uF
- C26: value 1uF -> 0.1uF
- C3: value 3.9pF -> 0.1uF
- C4: value 8.2pF -> 0.1uF
- C5, C6: value 100nF -> 0.1uF
- R1: value 56k -> (none)
- R5: value 10k -> (none)
- R6: value 63 -> (none)
Connections:
- removed net N$14: C29.2, U3.PA00(XIN32/SER1:0/TC2:0), Y2.2
- removed net N$15: C28.2, U3.PA01(XOUT32/SER1:1/TC2:1), Y2.1
- new net D+: IC2.USBDP, R9.1
- new net D-: IC2.USBDM, R8.1
- new net N$17: C37.1, JP2.D-, R8.2
- new net N$2: C36.1, JP2.D+, R9.2
- new net N$25: IC2.TXD
- new net N$26: IC2.RXD
- new net N$27: IC2.RTS#
- new net N$28: IC2.CTS#
- new net USB_VIN: IC2.VCC, JP2.VBUS
- net !RESET: now also TP3.TP; no longer JP1.!RESET
- net 3.3V: now also C10.2, C11.2, C12.2, C33.1, C6.2, C7.2, C9.2, R2.2, U$1.AVDD1, U$1.AVDD2, U$1.AVDD3, U$1.AVDD4, U$1.DGUARD, U$1.DVDD; no longer JP1.VCC, R3.1
- net CS_TX: now also R2.1; no longer R3.2
- net GND: now also C33.2, C34.-, C36.2, C37.2, IC2.GND, IC2.GND_EP, JP2.GND, JP2.SHIELD, TP4.TP; no longer C1.2, C15.-, C16.-, C2.2, C28.1, C29.1, JP1.GND@3, JP1.GND@5, U2.GND
- net RX: no longer JP1.SWO/TDO
- net SWCLK: now also TP1.TP; no longer JP1.SWDCLK/TCK
- net SWDIO: now also TP2.TP; no longer JP1.SWDIO/TMS
- net TX: no longer JP1.NC/TDI
- net VDD: now also IC2.3V3OUT, IC2.RESET#, IC2.VCCIO; no longer C10.2, C11.2, C12.2, C15.+, C2.1, C6.2, C7.2, C9.2, U$1.AVDD1, U$1.AVDD2, U$1.AVDD3, U$1.AVDD4, U$1.DGUARD, U$1.DVDD, U2.OUT
- net V_BATT: now also C34.+; no longer C1.1, C16.+, U2.EN, U2.IN
Other:
- moved on the sheet: C10, C11, C12, C13, C14, C17, C18, C19, C20, C21, C22, C23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

Commit message: tracker board work
Connections:
- removed net N$25: IC2.TXD
- removed net N$26: IC2.RXD
- removed net N$27: IC2.RTS#
- removed net N$28: IC2.CTS#
- new net CTS: IC2.CTS#, U3.PA15(XOUT/SER2:3+)
- new net RTS: IC2.RTS#, U3.PA14(XIN/SER2:2+)
- new net RXD: IC2.TXD, U3.PA13(I2C/SER2:1+)
- new net TXD: IC2.RXD, U3.PA12(I2C/SER2:0+)
- net LED: no longer U3.PA15(XOUT/SER2:3+)
Changed lines of the file:
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@@
 <label x="246.38" y="25.4" size="1.27" layer="95" rot="R90" xref="yes"/>
-</segment>
-<segment>
-<pinref part="U3" gate="G$1" pin="PA15(XOUT/SER2:3+)"/>
-<wire x1="218.44" y1="58.42" x2="220.98" y2="58.42" width="0.1524" layer="91"/>
-<label x="220.98" y="58.42" size="1.27" layer="95" xref="yes"/>
 </segment>
 </net>
@@
 </segment>
 </net>
-<net name="N$25" class="0">
-<segment>
-<pinref part="IC2" gate="G$1" pin="TXD"/>
-<wire x1="2.54" y1="223.52" x2="5.08" y2="223.52" width="0.1524" layer="91"/>
-</segment>
-</net>
-<net name="N$26" class="0">
-<segment>
-<pinref part="IC2" gate="G$1" pin="RXD"/>
-<wire x1="2.54" y1="220.98" x2="5.08" y2="220.98" width="0.1524" layer="91"/>
-</segment>
-</net>
-<net name="N$27" class="0">
-<segment>
-<pinref part="IC2" gate="G$1" pin="RTS#"/>
-<wire x1="2.54" y1="218.44" x2="5.08" y2="218.44" width="0.1524" layer="91"/>
-</segment>
-</net>
-<net name="N$28" class="0">
-<segment>
-<pinref part="IC2" gate="G$1" pin="CTS#"/>
-<wire x1="2.54" y1="215.9" x2="5.08" y2="215.9" width="0.1524" layer="91"/>
-</segment>
-</net>
 <net name="USB_VIN" class="0">
 <segment>
@@
 </segment>
 </net>
+<net name="CTS" class="0">
+<segment>
+<pinref part="U3" gate="G$1" pin="PA15(XOUT/SER2:3+)"/>
+<wire x1="218.44" y1="58.42" x2="220.98" y2="58.42" width="0.1524" layer="91"/>
+<label x="220.98" y="58.42" size="1.27" layer="95" xref="yes"/>
+</segment>
+<segment>
+<pinref part="IC2" gate="G$1" pin="CTS#"/>
+<wire x1="2.54" y1="215.9" x2="5.08" y2="215.9" width="0.1524" layer="91"/>
+<label x="5.08" y="215.9" size="1.27" layer="95" xref="yes"/>
+</segment>
+</net>
+<net name="RTS" class="0">
+<segment>
+<pinref part="U3" gate="G$1" pin="PA14(XIN/SER2:2+)"/>
+<wire x1="218.44" y1="60.96" x2="220.98" y2="60.96" width="0.1524" layer="91"/>
+<label x="220.98" y="60.96" size="1.27" layer="95" xref="yes"/>
+</segment>
+<segment>
+<pinref part="IC2" gate="G$1" pin="RTS#"/>
+<wire x1="2.54" y1="218.44" x2="5.08" y2="218.44" width="0.1524" layer="91"/>
+<label x="5.08" y="218.44" size="1.27" layer="95" xref="yes"/>
+</segment>
+</net>
+<net name="RXD" class="0">
+<segment>
+<pinref part="U3" gate="G$1" pin="PA13(I2C/SER2:1+)"/>
+<wire x1="218.44" y1="63.5" x2="220.98" y2="63.5" width="0.1524" layer="91"/>
+<label x="220.98" y="63.5" size="1.27" layer="95" xref="yes"/>
+</segment>
+<segment>
+<pinref part="IC2" gate="G$1" pin="TXD"/>
+<wire x1="2.54" y1="223.52" x2="5.08" y2="223.52" width="0.1524" layer="91"/>
+<label x="5.08" y="223.52" size="1.27" layer="95" xref="yes"/>
+</segment>
+</net>
+<net name="TXD" class="0">
+<segment>
+<pinref part="U3" gate="G$1" pin="PA12(I2C/SER2:0+)"/>
+<wire x1="218.44" y1="66.04" x2="220.98" y2="66.04" width="0.1524" layer="91"/>
+<label x="220.98" y="66.04" size="1.27" layer="95" xref="yes"/>
+</segment>
+<segment>
+<pinref part="IC2" gate="G$1" pin="RXD"/>
+<wire x1="2.54" y1="220.98" x2="5.08" y2="220.98" width="0.1524" layer="91"/>
+<label x="5.08" y="220.98" size="1.27" layer="95" xref="yes"/>
+</segment>
+</net>

Commit message: tracker work
Parts:
- removed TP1, TP2, TP3, TP4: TPSQTP06R, testpad:TPSQTP06R
- added JP1: CORTEX_DEBUG_PTH, SparkFun-Connectors:CORTEX_DEBUG_PTH
Connections:
- removed net AMP_EM: U1.EN, U3.PB23(SER5:3+)
- removed net VDD: IC2.3V3OUT, IC2.RESET#, IC2.VCCIO
- new net AMP_EN: U1.EN, U3.PA24(SER3:2+)
- net !RESET: now also JP1.!RESET; no longer TP3.TP
- net 3.3V: now also IC2.3V3OUT, IC2.RESET#, IC2.VCCIO, JP1.VCC
- net GND: now also JP1.GND@3, JP1.GND@5; no longer TP4.TP
- net RX: now also JP1.SWO/TDO, U3.PB23(SER5:3+); no longer U3.PA25(SER3:3+)
- net SER5_RX: no longer U3.PB03(AIN11/SER5:1)
- net SER5_TX: no longer U3.PB02(AIN10/SER5:0)
- net SWCLK: now also JP1.SWDCLK/TCK; no longer TP1.TP
- net SWDIO: now also JP1.SWDIO/TMS; no longer TP2.TP
- net TX: now also JP1.NC/TDI, U3.PB22(SER5:2+); no longer U3.PA24(SER3:2+)

Commit message: square mock up
Connections:
- removed net SER5_RX: IC1.TXD
- removed net SER5_TX: IC1.RXD
- new net GPS_RX: IC1.TXD, U3.PA01(XOUT32/SER1:1/TC2:1)
- new net GPS_TX: IC1.RXD, U3.PA00(XIN32/SER1:0/TC2:0)
- net LED: now also U3.PB09(AIN3/SER4:1/TC4:1)
Changed lines of the file:
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@@
 <?xml version="1.0" encoding="utf-8"?>
 <!DOCTYPE eagle SYSTEM "eagle.dtd">
-<eagle version="8.5.0">
+<eagle version="8.6.0">
 <drawing>
 <settings>
@@
 <instance part="SUPPLY10" gate="G$1" x="127" y="93.98"/>
 <instance part="SUPPLY11" gate="G$1" x="134.62" y="93.98"/>
-<instance part="SUPPLY12" gate="G$1" x="147.32" y="93.98"/>
+<instance part="SUPPLY12" gate="G$1" x="147.32" y="96.52"/>
 <instance part="SUPPLY13" gate="G$1" x="220.98" y="91.44"/>
 <instance part="SUPPLY17" gate="G$1" x="93.98" y="101.6"/>
@@
 <label x="246.38" y="25.4" size="1.27" layer="95" rot="R90" xref="yes"/>
 </segment>
+<segment>
+<pinref part="U3" gate="G$1" pin="PB09(AIN3/SER4:1/TC4:1)"/>
+<wire x1="149.86" y1="25.4" x2="147.32" y2="25.4" width="0.1524" layer="91"/>
+<label x="147.32" y="25.4" size="1.27" layer="95" rot="R180" xref="yes"/>
+</segment>
 </net>
 <net name="SWCLK" class="0">
@@
 <pinref part="R4" gate="G$1" pin="2"/>
 <pinref part="SUPPLY12" gate="G$1" pin="3.3V"/>
+<wire x1="147.32" y1="96.52" x2="147.32" y2="93.98" width="0.1524" layer="91"/>
 </segment>
 <segment>
@@
 </segment>
 </net>
-<net name="SER5_TX" class="0">
-<segment>
-<pinref part="IC1" gate="G$1" pin="RXD"/>
-<wire x1="38.1" y1="139.7" x2="43.18" y2="139.7" width="0.1524" layer="91"/>
-<label x="43.18" y="139.7" size="1.27" layer="95" xref="yes"/>
-</segment>
-</net>
-<net name="SER5_RX" class="0">
-<segment>
-<pinref part="IC1" gate="G$1" pin="TXD"/>
-<wire x1="38.1" y1="137.16" x2="43.18" y2="137.16" width="0.1524" layer="91"/>
-<label x="43.18" y="137.16" size="1.27" layer="95" xref="yes"/>
-</segment>
-</net>
 <net name="TX_MOSI" class="0">
 <segment>
@@
 </segment>
 </net>
+<net name="GPS_TX" class="0">
+<segment>
+<pinref part="U3" gate="G$1" pin="PA00(XIN32/SER1:0/TC2:0)"/>
+<wire x1="149.86" y1="55.88" x2="147.32" y2="55.88" width="0.1524" layer="91"/>
+<label x="147.32" y="55.88" size="1.27" layer="95" rot="R180" xref="yes"/>
+</segment>
+<segment>
+<pinref part="IC1" gate="G$1" pin="RXD"/>
+<wire x1="38.1" y1="139.7" x2="43.18" y2="139.7" width="0.1524" layer="91"/>
+<label x="43.18" y="139.7" size="1.27" layer="95" xref="yes"/>
+</segment>
+</net>
+<net name="GPS_RX" class="0">
+<segment>
+<pinref part="U3" gate="G$1" pin="PA01(XOUT32/SER1:1/TC2:1)"/>
+<wire x1="149.86" y1="50.8" x2="147.32" y2="50.8" width="0.1524" layer="91"/>
+<label x="147.32" y="50.8" size="1.27" layer="95" rot="R180" xref="yes"/>
+</segment>
+<segment>
+<pinref part="IC1" gate="G$1" pin="TXD"/>
+<wire x1="38.1" y1="137.16" x2="43.18" y2="137.16" width="0.1524" layer="91"/>
+<label x="43.18" y="137.16" size="1.27" layer="95" xref="yes"/>
+</segment>
+</net>

Commit message: test flight three
Parts:
- C10, C22, C7: value 0.1uF -> 10nF
- C11, C12, C9: value 0.1uF -> 220pF
- C17, C21: value 0.1uF -> 220pf
- C19: value 0.1uF -> 8.2pF
- C20: value 0.1uF -> 5.6pF
- C26: value 0.1uF -> 1uF
- C3, C4: value 0.1uF -> 3.9pF
- L2: value 6.8NH -> 27NH
- L4: value 6.8NH -> 22NH
Changed lines of the file:
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@@
 <?xml version="1.0" encoding="utf-8"?>
 <!DOCTYPE eagle SYSTEM "eagle.dtd">
-<eagle version="8.6.0">
+<eagle version="8.7.0">
 <drawing>
 <settings>
@@
 <part name="C5" library="SparkFun-Capacitors" deviceset="0.1UF" device="-0402-16V-10%" value="0.1uF"/>
 <part name="C6" library="SparkFun-Capacitors" deviceset="0.1UF" device="-0402-16V-10%" value="0.1uF"/>
-<part name="C7" library="SparkFun-Capacitors" deviceset="0.1UF" device="-0402-16V-10%" value="0.1uF"/>
-<part name="C9" library="SparkFun-Capacitors" deviceset="0.1UF" device="-0402-16V-10%" value="0.1uF"/>
-<part name="C10" library="SparkFun-Capacitors" deviceset="0.1UF" device="-0402-16V-10%" value="0.1uF"/>
-<part name="C11" library="SparkFun-Capacitors" deviceset="0.1UF" device="-0402-16V-10%" value="0.1uF"/>
-<part name="C12" library="SparkFun-Capacitors" deviceset="0.1UF" device="-0402-16V-10%" value="0.1uF"/>
+<part name="C7" library="SparkFun-Capacitors" deviceset="0.1UF" device="-0402-16V-10%" value="10nF"/>
+<part name="C9" library="SparkFun-Capacitors" deviceset="0.1UF" device="-0402-16V-10%" value="220pF"/>
+<part name="C10" library="SparkFun-Capacitors" deviceset="0.1UF" device="-0402-16V-10%" value="10nF"/>
+<part name="C11" library="SparkFun-Capacitors" deviceset="0.1UF" device="-0402-16V-10%" value="220pF"/>
+<part name="C12" library="SparkFun-Capacitors" deviceset="0.1UF" device="-0402-16V-10%" value="220pF"/>
 <part name="R1" library="SparkFun-Resistors" deviceset="RESISTOR" device="0402" value=" "/>
 <part name="Y1" library="SparkFun-Clocks" library_urn="urn:adsk.eagle:library:511" deviceset="CRYSTAL" device="SMD-3.2X2.5" package3d_urn="urn:adsk.eagle:package:37521/1" value="26MHz"/>
@@
 <part name="GND11" library="SparkFun-Aesthetics" deviceset="GND" device=""/>
 <part name="GND19" library="SparkFun-Aesthetics" deviceset="GND" device=""/>
-<part name="L2" library="SparkFun-Coils" library_urn="urn:adsk.eagle:library:512" deviceset="INDUCTOR" device="-0402-3.9NH" package3d_urn="urn:adsk.eagle:package:37575/1" value="6.8NH"/>
-<part name="C3" library="SparkFun-Capacitors" deviceset="0.1UF" device="-0402-16V-10%" value="0.1uF"/>
-<part name="C4" library="SparkFun-Capacitors" deviceset="0.1UF" device="-0402-16V-10%" value="0.1uF"/>
-<part name="C17" library="SparkFun-Capacitors" deviceset="0.1UF" device="-0402-16V-10%" value="0.1uF"/>
-<part name="C19" library="SparkFun-Capacitors" deviceset="0.1UF" device="-0402-16V-10%" value="0.1uF"/>
-<part name="C20" library="SparkFun-Capacitors" deviceset="0.1UF" device="-0402-16V-10%" value="0.1uF"/>
-<part name="C21" library="SparkFun-Capacitors" deviceset="0.1UF" device="-0402-16V-10%" value="0.1uF"/>
+<part name="L2" library="SparkFun-Coils" library_urn="urn:adsk.eagle:library:512" deviceset="INDUCTOR" device="-0402-3.9NH" package3d_urn="urn:adsk.eagle:package:37575/1" value="27NH"/>
+<part name="C3" library="SparkFun-Capacitors" deviceset="0.1UF" device="-0402-16V-10%" value="3.9pF"/>
+<part name="C4" library="SparkFun-Capacitors" deviceset="0.1UF" device="-0402-16V-10%" value="3.9pF"/>
+<part name="C17" library="SparkFun-Capacitors" deviceset="0.1UF" device="-0402-16V-10%" value="220pf"/>
+<part name="C19" library="SparkFun-Capacitors" deviceset="0.1UF" device="-0402-16V-10%" value="8.2pF"/>
+<part name="C20" library="SparkFun-Capacitors" deviceset="0.1UF" device="-0402-16V-10%" value="5.6pF"/>
+<part name="C21" library="SparkFun-Capacitors" deviceset="0.1UF" device="-0402-16V-10%" value="220pf"/>
 <part name="L1" library="SparkFun-Coils" library_urn="urn:adsk.eagle:library:512" deviceset="INDUCTOR" device="-0402-3.9NH" package3d_urn="urn:adsk.eagle:package:37575/1" value="27NH"/>
 <part name="L3" library="SparkFun-Coils" library_urn="urn:adsk.eagle:library:512" deviceset="INDUCTOR" device="-0402-3.9NH" package3d_urn="urn:adsk.eagle:package:37575/1" value="27NH"/>
-<part name="L4" library="SparkFun-Coils" library_urn="urn:adsk.eagle:library:512" deviceset="INDUCTOR" device="-0402-3.9NH" package3d_urn="urn:adsk.eagle:package:37575/1" value="6.8NH"/>
+<part name="L4" library="SparkFun-Coils" library_urn="urn:adsk.eagle:library:512" deviceset="INDUCTOR" device="-0402-3.9NH" package3d_urn="urn:adsk.eagle:package:37575/1" value="22NH"/>
 <part name="GND3" library="SparkFun-Aesthetics" deviceset="GND" device=""/>
 <part name="GND13" library="SparkFun-Aesthetics" deviceset="GND" device=""/>
@@
 <part name="GND21" library="SparkFun-Aesthetics" deviceset="GND" device=""/>
 <part name="L5" library="SparkFun-Coils" library_urn="urn:adsk.eagle:library:512" deviceset="INDUCTOR" device="-0402-3.9NH" package3d_urn="urn:adsk.eagle:package:37575/1" value="36nH"/>
-<part name="C22" library="SparkFun-Capacitors" deviceset="0.1UF" device="-0402-16V-10%" value="0.1uF"/>
+<part name="C22" library="SparkFun-Capacitors" deviceset="0.1UF" device="-0402-16V-10%" value="10nF"/>
 <part name="GND23" library="SparkFun-Aesthetics" deviceset="GND" device=""/>
 <part name="L6" library="SparkFun-Coils" library_urn="urn:adsk.eagle:library:512" deviceset="INDUCTOR" device="-0402-3.9NH" package3d_urn="urn:adsk.eagle:package:37575/1" value="51nH"/>
@@
 <part name="GND26" library="SparkFun-PowerSymbols" deviceset="GND" device=""/>
 <part name="C25" library="SparkFun-Capacitors" deviceset="0.1UF" device="-0402-16V-10%" value="0.1uF"/>
-<part name="C26" library="SparkFun-Capacitors" deviceset="0.1UF" device="-0402-16V-10%" value="0.1uF"/>
+<part name="C26" library="SparkFun-Capacitors" deviceset="0.1UF" device="-0402-16V-10%" value="1uF"/>
 <part name="C27" library="SparkFun-Capacitors" deviceset="0.1UF" device="-0402-16V-10%" value="0.1uF"/>
 <part name="U3" library="SparkFun-IC-Microcontroller" deviceset="ATSAMD21G" device="-A"/>
@@
 <instance part="C27" gate="G$1" x="127" y="55.88" smashed="yes">
 <attribute name="NAME" x="128.524" y="58.801" size="1.778" layer="95" font="vector"/>
-<attribute name="VALUE" x="120.904" y="53.721" size="1.778" layer="96" font="vector"/>
+<attribute name="VALUE" x="128.524" y="53.721" size="1.778" layer="96" font="vector"/>
 </instance>
 <instance part="U3" gate="G$1" x="182.88" y="40.64"/>
@@
 <instance part="R8" gate="G$1" x="-5.08" y="264.16" smashed="yes" rot="R180">
 <attribute name="NAME" x="-1.27" y="262.6614" size="1.27" layer="95" rot="R180"/>
-<attribute name="VALUE" x="-6.35" y="267.462" size="1.27" layer="96" rot="R180"/>
+<attribute name="VALUE" x="-3.81" y="259.842" size="1.27" layer="96" rot="R180"/>
 </instance>
 <instance part="R9" gate="G$1" x="-5.08" y="261.62" smashed="yes" rot="R180">
 <attribute name="NAME" x="-1.27" y="260.1214" size="1.27" layer="95" rot="R180"/>
-<attribute name="VALUE" x="-6.35" y="264.922" size="1.27" layer="96" rot="R180"/>
+<attribute name="VALUE" x="-3.81" y="267.462" size="1.27" layer="96" rot="R180"/>
 </instance>
 <instance part="SUPPLY14" gate="G$1" x="101.6" y="228.6"/>
