File: DasAltimeter V0.35/DasAltimeter V0.35/DasAltimeter V0.35.brd (EAGLE design)
At the start: 38.9 x 21.6 mm, 56 parts, among them IC1 BMI055, U1 ATSAMD21G-A, U2 3.3V/150mA, U3 MS5803-14BA, U5 ADXL377, X1 22-23-2041, X2 22-23-2041

Commit message: routed dasAltimeter V0.40 and updates to code
Parts:
- added U$5: STM32F405RGT6, SparkFun-IC-Microcontroller:TQFP64
Changed lines of the file:
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@@
 <?xml version="1.0" encoding="utf-8"?>
 <!DOCTYPE eagle SYSTEM "eagle.dtd">
-<eagle version="8.7.0">
+<eagle version="9.5.2">
 <drawing>
 <settings>
@@
 <param name="checkStop" value="0"/>
 <param name="checkValues" value="0"/>
+<param name="checkNames" value="1"/>
+<param name="checkWireStubs" value="1"/>
+<param name="checkPolygonWidth" value="0"/>
 <param name="useDiameter" value="13"/>
 <param name="maxErrors" value="50"/>
@@
 <attribute name="PROD_ID" value="DIO-00862" x="34.544" y="6.731" size="1.778" layer="28" rot="MR270" display="off"/>
 </element>
-<element name="FRAME1" library="SparkFun-Aesthetics" package="DUMMY" value="FRAME-LETTERNO_PACKAGE" x="-24.13" y="48.26">
+<element name="FRAME1" library="SparkFun-Aesthetics" package="DUMMY" value="FRAME-LETTERNO_PACKAGE" x="-24.13" y="48.26" smashed="yes">
 <attribute name="DESIGNER" value="Nobody" x="-24.13" y="48.26" size="1.778" layer="27" display="off"/>
 <attribute name="VERSION" value="v01" x="-24.13" y="48.26" size="1.778" layer="27" display="off"/>
@@
 <attribute name="PROD_ID" value="NDUC-07874" x="15.0495" y="-0.127" size="1.778" layer="27" rot="R180" display="off"/>
 </element>
-<element name="R1" library="SparkFun-Resistors" package="0402" value="10k" x="24.384" y="14.478" rot="R180">
+<element name="R1" library="SparkFun-Resistors" package="0402" value="10k" x="24.384" y="14.478" smashed="yes" rot="R180">
+<attribute name="NAME" x="24.384" y="13.716" size="0.6096" layer="25" font="vector" ratio="20" rot="R180" align="bottom-center"/>
 <attribute name="PROD_ID" value=" " x="24.384" y="14.478" size="1.778" layer="27" rot="R180" display="off"/>
+<attribute name="VALUE" x="24.384" y="15.24" size="0.6096" layer="27" font="vector" ratio="20" rot="R180" align="top-center"/>
 </element>
 <element name="R10" library="SparkFun-Resistors" package="0402" value="27k" x="10.922" y="4.191" smashed="yes" rot="R180">
@@
 <attribute name="PROD_ID" value="COMP-08568" x="30.226" y="12.7" size="1.778" layer="28" rot="MR180" display="off"/>
 </element>
-<element name="U$1" library="SaL-lib1" package="PB-5R0H104-R" value="PB-5R0H104-R" x="12.573" y="11.684" rot="MR180"/>
+<element name="U$1" library="SaL-lib1" package="PB-5R0H104-R" value="PB-5R0H104-R" x="12.573" y="11.684" smashed="yes" rot="MR180"/>
 <element name="U1" library="SparkFun-IC-Microcontroller" package="TQFP-48" value="ATSAMD21G-A" x="19.558" y="7.62" smashed="yes" rot="R45">
 <attribute name="PROD_ID" value="IC-13064" x="19.558" y="7.62" size="1.778" layer="27" rot="R45" display="off"/>
@@
 <attribute name="PROD_ID" value="IC-12111" x="29.083" y="6.096" size="1.778" layer="27" rot="R270" display="off"/>
 </element>
-<element name="X1" library="con-molex" library_urn="urn:adsk.eagle:library:165" package="22-23-2041" value="22-23-2041" x="8.001" y="0.508" smashed="yes" rot="MR0">
+<element name="X1" library="con-molex" library_urn="urn:adsk.eagle:library:165" package="22-23-2041" package3d_urn="urn:adsk.eagle:package:8078635/1" value="22-23-2041" x="8.001" y="0.508" smashed="yes" rot="MR0">
 <attribute name="MF" value="MOLEX" x="8.001" y="0.508" size="1.778" layer="28" rot="MR0" display="off"/>
 <attribute name="MPN" value="22-23-2041" x="8.001" y="0.508" size="1.778" layer="28" rot="MR0" display="off"/>
 <attribute name="OC_FARNELL" value="1462920" x="8.001" y="0.508" size="1.778" layer="28" rot="MR0" display="off"/>
 <attribute name="OC_NEWARK" value="38C0355" x="8.001" y="0.508" size="1.778" layer="28" rot="MR0" display="off"/>
-</element>
-<element name="X2" library="con-molex" library_urn="urn:adsk.eagle:library:165" package="22-23-2041" value="22-23-2041" x="8.001" y="15.494" smashed="yes" rot="MR180">
+<attribute name="POPULARITY" value="21" x="8.001" y="0.508" size="1.778" layer="28" rot="MR0" display="off"/>
+</element>
+<element name="X2" library="con-molex" library_urn="urn:adsk.eagle:library:165" package="22-23-2041" package3d_urn="urn:adsk.eagle:package:8078635/1" value="22-23-2041" x="8.001" y="15.494" smashed="yes" rot="MR180">
 <attribute name="MF" value="MOLEX" x="8.001" y="15.494" size="1.778" layer="28" rot="MR180" display="off"/>
 <attribute name="MPN" value="22-23-2041" x="8.001" y="15.494" size="1.778" layer="28" rot="MR180" display="off"/>
 <attribute name="OC_FARNELL" value="1462920" x="8.001" y="15.494" size="1.778" layer="28" rot="MR180" display="off"/>
 <attribute name="OC_NEWARK" value="38C0355" x="8.001" y="15.494" size="1.778" layer="28" rot="MR180" display="off"/>
+<attribute name="POPULARITY" value="21" x="8.001" y="15.494" size="1.778" layer="28" rot="MR180" display="off"/>
 </element>
 <element name="H1" library="SparkFun-Hardware" package="STAND-OFF-TIGHT" value="STAND-OFFTIGHT" x="0" y="16.002" smashed="yes"/>
@@
 </element>
 <element name="U$2" library="SaL-lib1" package="AT25SF081" value="AT25SF081" x="29.083" y="14.605" smashed="yes" rot="R270"/>
-<element name="J1" library="SparkFun-Connectors" library_urn="urn:adsk.eagle:library:513" package="1X02_2.54_SCREWTERM" package3d_urn="urn:adsk.eagle:package:38059/1" value="" x="0.6985" y="6.731" rot="MR90"/>
+<element name="J1" library="SparkFun-Connectors" library_urn="urn:adsk.eagle:library:513" package="1X02_2.54_SCREWTERM" package3d_urn="urn:adsk.eagle:package:38059/1" value="" x="0.6985" y="6.731" smashed="yes" rot="MR90">
+<attribute name="NAME" x="4.1275" y="5.461" size="0.6096" layer="26" font="vector" ratio="20" rot="MR90"/>
+<attribute name="VALUE" x="-3.3655" y="5.461" size="0.6096" layer="28" font="vector" ratio="20" rot="MR90"/>
+</element>
 <element name="C7" library="SparkFun-Capacitors" package="0402" value="100nF" x="26.6065" y="17.018" smashed="yes" rot="R90">
 <attribute name="NAME" x="27.686" y="15.1765" size="0.6096" layer="25" font="vector" ratio="20" rot="R90" align="bottom-center"/>
 <attribute name="PROD_ID" value="CAP-12416" x="26.6065" y="17.018" size="1.778" layer="27" rot="R90" display="off"/>
+</element>
+<element name="U$5" library="SparkFun-IC-Microcontroller" package="TQFP64" value="STM32F405RGT6" x="-12.7" y="7.62" smashed="yes">
+<attribute name="NAME" x="-19.685" y="7.62" size="0.6096" layer="25" font="vector" ratio="20" rot="R90" align="bottom-center"/>
+<attribute name="PROD_ID" value="IC-11709" x="-12.7" y="7.62" size="1.778" layer="27" display="off"/>
+<attribute name="VALUE" x="-5.08" y="7.62" size="0.6096" layer="27" font="vector" ratio="20" rot="R90" align="bottom-center"/>
 </element>
 </elements>
@@
 </signal>
 </signals>
+<mfgpreviewcolors>
+<mfgpreviewcolor name="soldermaskcolor" color="0xC8008000"/>
+<mfgpreviewcolor name="silkscreencolor" color="0xFFFEFEFE"/>
+<mfgpreviewcolor name="backgroundcolor" color="0xFF282828"/>
+<mfgpreviewcolor name="coppercolor" color="0xFFFFBF00"/>
+<mfgpreviewcolor name="substratecolor" color="0xFF786E46"/>
+</mfgpreviewcolors>
 </board>
 </drawing>
