File: DasAltimeter V0.42/DasAltimeter V0.41.brd (EAGLE design)
At the start: 38.9 x 21.6 mm, 57 parts, among them IC1 BMI055, IC2 MCP73811/2, U2 3.3V/150mA, U3 MS5803-14BA, U5 ADXL377, X1 22-23-2041, X2 22-23-2041

Commit message: lots of parabeep code updates, gps started
Parts:
- added J3: TC2030-IDC-NL, TC2030-IDC-NL:TAG_TC2030-IDC-NL
- added LS1: CMT-8503-87-SMT-TR, CMT-8503-87-SMT-TR:XDCR_CMT-8503-87-SMT-TR
- added LS2: CMT-4023S-SMT-TR, CMT-4023S-SMT-TR:CUI_CMT-4023S-SMT-TR
- L1: value FB 30Ohm -> 33nH/±5%/500mA
- R1, R23, R24, R4, R5: value 10k -> (none)
- R10, R14, R18, R22, R3: value 27k -> (none)
- R11, R15, R19, R7: value 100 -> (none)
- R12, R16, R20, R8: value 3.3k -> (none)
- R13, R17, R21, R6, R9: value 100k -> (none)
- R2, R25: value 63 -> (none)
- moved SG1 27.4 mm to (56.9, 6.35)
- moved D2 15.4 mm to (47.4, 13.7), turned to 0 degrees
- moved R2 10.2 mm to (39.1, 15.7)
Routing:
- net LED: track 12.7 -> 0.00 mm, vias 1 -> 0
- net BUZZER: track 5.73 -> 0.00 mm, vias 1 -> 0
- net N$29: track 2.32 -> 0.44 mm, vias 1 -> 0
- net GND: vias 38 -> 11
- removed copper zone on layer 15, net 3.3V
- removed copper zone on layer 1, net GND
- removed copper zone on layer 16, net GND
- removed copper zone on layer 2, net GND
Other:
- board size 38.9 x 21.6 mm -> 46.5 x 21.6 mm
