File: DasAltimeter V0.42/DasAltimeter V0.41.sch (EAGLE design)
At the start: 57 parts, among them IC1 BMI055, IC2 MCP73811/2, U2 3.3V/150mA, U3 MS5803-14BA, U5 ADXL377, X1 22-23-2041, X2 22-23-2041

Commit message: lots of parabeep code updates, gps started
Parts:
- added J3: TC2030-IDC-NL, TC2030-IDC-NL:TC2030-IDC-NL
- added LS1: CMT-8503-87-SMT-TR, CMT-8503-87-SMT-TR:CMT-8503-87-SMT-TR
- added LS2: CMT-4023S-SMT-TR, CMT-4023S-SMT-TR:CMT-4023S-SMT-TR
- L1: value FB 30Ohm -> 33nH/±5%/500mA
- R1, R23, R24, R4, R5: value 10k -> (none)
- R10, R14, R18, R22, R3: value 27k -> (none)
- R11, R15, R19, R7: value 100 -> (none)
- R12, R16, R20, R8: value 3.3k -> (none)
- R13, R17, R21, R6, R9: value 100k -> (none)
- R2, R25: value 63 -> (none)
Changed lines of the file:
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@@
 <part name="C9" library="SparkFun-Capacitors" deviceset="0.1UF" device="-0402-16V-10%" value="0.1uF"/>
 <part name="C10" library="SparkFun-Capacitors" deviceset="0.1UF" device="-0402-16V-10%" value="0.1uF"/>
-<part name="L1" library="SparkFun-Coils" deviceset="INDUCTOR" device="-0603-33NH" value="FB 30Ohm"/>
+<part name="L1" library="SparkFun-Coils" deviceset="INDUCTOR" device="-0603-33NH" value="33nH/±5%/500mA"/>
 <part name="C11" library="SparkFun-Capacitors" deviceset="0.1UF" device="-0402-16V-10%" value="0.1uF"/>
 <part name="GND15" library="SparkFun-Aesthetics" deviceset="GND" device=""/>
@@
 <part name="D2" library="SparkFun-LED" deviceset="LED-GREEN" device="1206" value="GREEN"/>
 <part name="GND51" library="SparkFun-Aesthetics" deviceset="GND" device=""/>
-<part name="R2" library="SparkFun-Resistors" deviceset="RESISTOR" device="0402" value="63"/>
-<part name="R3" library="SparkFun-Resistors" deviceset="RESISTOR" device="0402" value="27k"/>
+<part name="R2" library="SparkFun-Resistors" deviceset="RESISTOR" device="0402" value=" "/>
+<part name="R3" library="SparkFun-Resistors" deviceset="RESISTOR" device="0402" value=" "/>
 <part name="U3" library="SparkFun-Sensors" deviceset="MS5803-14BA" device=""/>
 <part name="SUPPLY9" library="SparkFun-Aesthetics" deviceset="3.3V" device=""/>
@@
 <part name="SUPPLY13" library="SparkFun-Aesthetics" deviceset="3.3V" device=""/>
 <part name="GND6" library="SparkFun-Aesthetics" deviceset="GND" device=""/>
-<part name="R4" library="SparkFun-Resistors" deviceset="RESISTOR" device="0402" value="10k"/>
+<part name="R4" library="SparkFun-Resistors" deviceset="RESISTOR" device="0402" value=" "/>
 <part name="GND7" library="SparkFun-Aesthetics" deviceset="GND" device=""/>
-<part name="R5" library="SparkFun-Resistors" deviceset="RESISTOR" device="0402" value="10k"/>
+<part name="R5" library="SparkFun-Resistors" deviceset="RESISTOR" device="0402" value=" "/>
 <part name="GND8" library="SparkFun-Aesthetics" deviceset="GND" device=""/>
 <part name="SUPPLY14" library="SparkFun-Aesthetics" deviceset="3.3V" device=""/>
-<part name="R6" library="SparkFun-Resistors" deviceset="RESISTOR" device="0402" value="100k"/>
-<part name="R7" library="SparkFun-Resistors" deviceset="RESISTOR" device="0402" value="100"/>
-<part name="R8" library="SparkFun-Resistors" deviceset="RESISTOR" device="0402" value="3.3k"/>
-<part name="R9" library="SparkFun-Resistors" deviceset="RESISTOR" device="0402" value="100k"/>
-<part name="R10" library="SparkFun-Resistors" deviceset="RESISTOR" device="0402" value="27k"/>
-<part name="R11" library="SparkFun-Resistors" deviceset="RESISTOR" device="0402" value="100"/>
-<part name="R12" library="SparkFun-Resistors" deviceset="RESISTOR" device="0402" value="3.3k"/>
-<part name="R13" library="SparkFun-Resistors" deviceset="RESISTOR" device="0402" value="100k"/>
-<part name="R14" library="SparkFun-Resistors" deviceset="RESISTOR" device="0402" value="27k"/>
-<part name="R15" library="SparkFun-Resistors" deviceset="RESISTOR" device="0402" value="100"/>
-<part name="R16" library="SparkFun-Resistors" deviceset="RESISTOR" device="0402" value="3.3k"/>
-<part name="R17" library="SparkFun-Resistors" deviceset="RESISTOR" device="0402" value="100k"/>
-<part name="R18" library="SparkFun-Resistors" deviceset="RESISTOR" device="0402" value="27k"/>
-<part name="R19" library="SparkFun-Resistors" deviceset="RESISTOR" device="0402" value="100"/>
-<part name="R20" library="SparkFun-Resistors" deviceset="RESISTOR" device="0402" value="3.3k"/>
-<part name="R21" library="SparkFun-Resistors" deviceset="RESISTOR" device="0402" value="100k"/>
-<part name="R22" library="SparkFun-Resistors" deviceset="RESISTOR" device="0402" value="27k"/>
+<part name="R6" library="SparkFun-Resistors" deviceset="RESISTOR" device="0402" value=" "/>
+<part name="R7" library="SparkFun-Resistors" deviceset="RESISTOR" device="0402" value=" "/>
+<part name="R8" library="SparkFun-Resistors" deviceset="RESISTOR" device="0402" value=" "/>
+<part name="R9" library="SparkFun-Resistors" deviceset="RESISTOR" device="0402" value=" "/>
+<part name="R10" library="SparkFun-Resistors" deviceset="RESISTOR" device="0402" value=" "/>
+<part name="R11" library="SparkFun-Resistors" deviceset="RESISTOR" device="0402" value=" "/>
+<part name="R12" library="SparkFun-Resistors" deviceset="RESISTOR" device="0402" value=" "/>
+<part name="R13" library="SparkFun-Resistors" deviceset="RESISTOR" device="0402" value=" "/>
+<part name="R14" library="SparkFun-Resistors" deviceset="RESISTOR" device="0402" value=" "/>
+<part name="R15" library="SparkFun-Resistors" deviceset="RESISTOR" device="0402" value=" "/>
+<part name="R16" library="SparkFun-Resistors" deviceset="RESISTOR" device="0402" value=" "/>
+<part name="R17" library="SparkFun-Resistors" deviceset="RESISTOR" device="0402" value=" "/>
+<part name="R18" library="SparkFun-Resistors" deviceset="RESISTOR" device="0402" value=" "/>
+<part name="R19" library="SparkFun-Resistors" deviceset="RESISTOR" device="0402" value=" "/>
+<part name="R20" library="SparkFun-Resistors" deviceset="RESISTOR" device="0402" value=" "/>
+<part name="R21" library="SparkFun-Resistors" deviceset="RESISTOR" device="0402" value=" "/>
+<part name="R22" library="SparkFun-Resistors" deviceset="RESISTOR" device="0402" value=" "/>
 <part name="X1" library="con-molex" library_urn="urn:adsk.eagle:library:165" deviceset="22-23-2041" device="" package3d_urn="urn:adsk.eagle:package:8078635/1"/>
 <part name="X2" library="con-molex" library_urn="urn:adsk.eagle:library:165" deviceset="22-23-2041" device="" package3d_urn="urn:adsk.eagle:package:8078635/1"/>
-<part name="R23" library="SparkFun-Resistors" deviceset="RESISTOR" device="0402" value="10k"/>
+<part name="R23" library="SparkFun-Resistors" deviceset="RESISTOR" device="0402" value=" "/>
 <part name="U$1" library="SaL-lib1" deviceset="PB-5R0H104-R" device=""/>
 <part name="IC1" library="BMI055" deviceset="BMI055" device=""/>
-<part name="R24" library="SparkFun-Resistors" deviceset="RESISTOR" device="0402" value="10k"/>
+<part name="R24" library="SparkFun-Resistors" deviceset="RESISTOR" device="0402" value=" "/>
 <part name="SUPPLY15" library="SparkFun-PowerSymbols" deviceset="3.3V" device=""/>
 <part name="GND10" library="SparkFun-PowerSymbols" deviceset="GND" device=""/>
@@
 <part name="GND9" library="SparkFun-Aesthetics" deviceset="GND" device=""/>
 <part name="SUPPLY5" library="SparkFun-PowerSymbols" deviceset="3.3V" device=""/>
-<part name="R1" library="SparkFun-Resistors" deviceset="RESISTOR" device="0402" value="10k"/>
+<part name="R1" library="SparkFun-Resistors" deviceset="RESISTOR" device="0402" value=" "/>
 <part name="IC2" library="adafruit" library_urn="urn:adsk.eagle:library:420" deviceset="MCP73811/2" device="" package3d_urn="urn:adsk.eagle:package:6240724/1"/>
 <part name="SUPPLY12" library="SparkFun-PowerSymbols" deviceset="VCC" device=""/>
 <part name="GND5" library="SparkFun-Aesthetics" deviceset="GND" device=""/>
-<part name="R25" library="SparkFun-Resistors" deviceset="RESISTOR" device="0402" value="63"/>
+<part name="R25" library="SparkFun-Resistors" deviceset="RESISTOR" device="0402" value=" "/>
 <part name="GND29" library="SparkFun-Aesthetics" deviceset="GND" device=""/>
+<part name="J3" library="TC2030-IDC-NL" deviceset="TC2030-IDC-NL" device=""/>
+<part name="LS1" library="CMT-8503-87-SMT-TR" deviceset="CMT-8503-87-SMT-TR" device=""/>
+<part name="LS2" library="CMT-4023S-SMT-TR" deviceset="CMT-4023S-SMT-TR" device=""/>
 </parts>
 <sheets>
@@
 <attribute name="VALUE" x="175.26" y="48.26" size="1.778" layer="96"/>
 </instance>
+<instance part="J3" gate="G$1" x="111.76" y="167.64" smashed="yes">
+<attribute name="NAME" x="106.67376875" y="180.3556" size="1.271559375" layer="95"/>
+<attribute name="VALUE" x="106.6798" y="157.4796" size="1.27005" layer="96"/>
+</instance>
+<instance part="LS1" gate="G$1" x="139.7" y="76.2" smashed="yes">
+<attribute name="NAME" x="135.89" y="85.09" size="1.778" layer="95"/>
+<attribute name="VALUE" x="135.89" y="66.04" size="1.778" layer="96" align="top-left"/>
+</instance>
+<instance part="LS2" gate="G$1" x="149.86" y="81.28" smashed="yes">
+<attribute name="NAME" x="146.04713125" y="90.1767" size="1.779340625" layer="95"/>
+<attribute name="VALUE" x="146.042409375" y="69.8272" size="1.781540625" layer="96"/>
+</instance>
 </instances>
