File: Parabeep V0.3/ParaBeep V0.3.brd (EAGLE design)
At the start: 35.3 x 57.5 mm, 64 parts, among them IC2 MCP73811/2, Q1 500mA/300V, U1 ADXL345, U2 TPS78330DDCRDDC5_TEX-L, U3 TPS78330DDCRDDC5_TEX-L, U4 UBLOX_SAM_M8Q-0-10, U5 MS5803-14BA, U6 ATSAMD51J20A-A, U7 AT25SF128A-SHB-T, U8 RN4871-V/RM118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

Commit message: bluetooth working, neeed usb c
Parts:
- R12: value (none) -> 64
- R13: value (none) -> 180
- R20, R29: value (none) -> 6.12M
- R21: value (none) -> 3.83M
- R22, R26: value (none) -> 5.62M
- R23, R24: value (none) -> 4.42M
- R25: value (none) -> 2k
- R27: value (none) -> 10M
- R28: value (none) -> 3.32M
- R30: value (none) -> 542K
- R5: value (none) -> 100k
