File: Parabeep V0.3/ParaBeep V0.3.sch (EAGLE design)
At the start: 63 parts, among them IC2 MCP73811/2, Q1 500mA/300V, U1 ADXL345, U2 TPS78330DDCRDDC5_TEX-L, U3 TPS78330DDCRDDC5_TEX-L, U4 UBLOX_SAM_M8Q-0-10, U5 MS5803-14BA, U6 ATSAMD51J20A-A, U7 AT25SF128A-SHB-T, U8 RN4871-V/RM118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

Commit message: bluetooth working, neeed usb c
Parts:
- R12: value (none) -> 64
- R13: value (none) -> 180
- R20, R29: value (none) -> 6.12M
- R21: value (none) -> 3.83M
- R22, R26: value (none) -> 5.62M
- R23, R24: value (none) -> 4.42M
- R25: value (none) -> 2k
- R27: value (none) -> 10M
- R28: value (none) -> 3.32M
- R30: value (none) -> 542K
- R5: value (none) -> 100k
Changed lines of the file:
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@@
 <part name="GND11" library="SparkFun-Aesthetics" deviceset="GND" device=""/>
 <part name="D1" library="SparkFun-DiscreteSemi" deviceset="DIODE" device="-BAS16J" value="250mA/100V"/>
-<part name="R13" library="SparkFun-Resistors" deviceset="RESISTOR" device="0402" value=" "/>
+<part name="R13" library="SparkFun-Resistors" deviceset="RESISTOR" device="0402" value="180"/>
 <part name="SUPPLY5" library="SparkFun-PowerSymbols" deviceset="VCC_1" device=""/>
 <part name="C12" library="SparkFun-Capacitors" deviceset="0.1UF" device="-0603-25V-(+80/-20%)" value="10uF"/>
 <part name="L2" library="SparkFun-Coils" deviceset="INDUCTOR" device="FB-30OHM"/>
-<part name="R5" library="SparkFun-Resistors" deviceset="RESISTOR" device="0402" value=" "/>
+<part name="R5" library="SparkFun-Resistors" deviceset="RESISTOR" device="0402" value="100k"/>
 <part name="GND4" library="SparkFun-Aesthetics" deviceset="GND" device=""/>
 <part name="SUPPLY10" library="SparkFun-PowerSymbols" deviceset="VCC_1" device=""/>
@@
 <part name="IC2" library="adafruit" library_urn="urn:adsk.eagle:library:420" deviceset="MCP73811/2" device="" package3d_urn="urn:adsk.eagle:package:6240724/1"/>
 <part name="GND22" library="SparkFun-Aesthetics" deviceset="GND" device=""/>
-<part name="R25" library="SparkFun-Resistors" deviceset="RESISTOR" device="0402" value=" "/>
+<part name="R25" library="SparkFun-Resistors" deviceset="RESISTOR" device="0402" value="2k"/>
 <part name="GND29" library="SparkFun-Aesthetics" deviceset="GND" device=""/>
 <part name="SUPPLY14" library="SparkFun-PowerSymbols" deviceset="VIN" device=""/>
 <part name="D2" library="SparkFun-LED" deviceset="LED-GREEN" device="0603" value="GREEN"/>
-<part name="R12" library="SparkFun-Resistors" deviceset="RESISTOR" device="0402" value=" "/>
+<part name="R12" library="SparkFun-Resistors" deviceset="RESISTOR" device="0402" value="64"/>
 <part name="GND23" library="SparkFun-Aesthetics" deviceset="GND" device=""/>
 <part name="U$6" library="SparkFun-PowerSymbols" deviceset="VCC-ISO" device=""/>
@@
 <part name="GND30" library="SparkFun-Aesthetics" deviceset="GND" device=""/>
 <part name="GND31" library="SparkFun-Aesthetics" deviceset="GND" device=""/>
-<part name="R20" library="SparkFun-Resistors" deviceset="RESISTOR" device="0402" value=" "/>
-<part name="R21" library="SparkFun-Resistors" deviceset="RESISTOR" device="0402" value=" "/>
-<part name="R22" library="SparkFun-Resistors" deviceset="RESISTOR" device="0402" value=" "/>
-<part name="R23" library="SparkFun-Resistors" deviceset="RESISTOR" device="0402" value=" "/>
-<part name="R24" library="SparkFun-Resistors" deviceset="RESISTOR" device="0402" value=" "/>
-<part name="R26" library="SparkFun-Resistors" deviceset="RESISTOR" device="0402" value=" "/>
-<part name="R27" library="SparkFun-Resistors" deviceset="RESISTOR" device="0402" value=" "/>
-<part name="R28" library="SparkFun-Resistors" deviceset="RESISTOR" device="0402" value=" "/>
-<part name="R29" library="SparkFun-Resistors" deviceset="RESISTOR" device="0402" value=" "/>
-<part name="R30" library="SparkFun-Resistors" deviceset="RESISTOR" device="0402" value=" "/>
+<part name="R20" library="SparkFun-Resistors" deviceset="RESISTOR" device="0402" value="6.12M"/>
+<part name="R21" library="SparkFun-Resistors" deviceset="RESISTOR" device="0402" value="3.83M"/>
+<part name="R22" library="SparkFun-Resistors" deviceset="RESISTOR" device="0402" value="5.62M"/>
+<part name="R23" library="SparkFun-Resistors" deviceset="RESISTOR" device="0402" value="4.42M"/>
+<part name="R24" library="SparkFun-Resistors" deviceset="RESISTOR" device="0402" value="4.42M"/>
+<part name="R26" library="SparkFun-Resistors" deviceset="RESISTOR" device="0402" value="5.62M"/>
+<part name="R27" library="SparkFun-Resistors" deviceset="RESISTOR" device="0402" value="10M"/>
+<part name="R28" library="SparkFun-Resistors" deviceset="RESISTOR" device="0402" value="3.32M"/>
+<part name="R29" library="SparkFun-Resistors" deviceset="RESISTOR" device="0402" value="6.12M"/>
+<part name="R30" library="SparkFun-Resistors" deviceset="RESISTOR" device="0402" value="542K"/>
 <part name="L4" library="SparkFun-Coils" deviceset="INDUCTOR" device="-CDRH-4.7UH" value="22µH - 744031220"/>
 <part name="C24" library="SparkFun-Capacitors" deviceset="4.7UF" device="-0603-6.3V-(10%)" value="4.7uF"/>
