File: ParaBeep V0.35B/ParaBeep V0.35.sch (EAGLE design)
At the start: 64 parts, among them IC2 MCP73811/2, Q1 500mA/300V, U1 ADXL345, U2 TPS78330DDCRDDC5_TEX-L, U3 TPS78330DDCRDDC5_TEX-L, U4 UBLOX_SAM_M8Q-0-10, U5 MS5803-14BA, U6 ATSAMD51J20A-A, U7 AT25SF128A-SHB-T, U8 RN4871-V/RM118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

Commit message: bluetooth working, usb next
Parts:
- removed J2: (no value), SparkFun-Connectors:USB_MICRO-B_FEMALE-SMT
- removed U7: AT25SF128A-SHB-T, AT25SF128A-SHB-T:AT25SF128A-SHB-T
- added C19: 10uF, SparkFun-Capacitors:10UF-POLAR-EIA3216-16V-10%(TANT)
- added J4: (no value), SparkFun-Connectors:USB_C_2-LAYER_PADS
- added JP2: JUMPER-SMT_3_1-NC_TRACE_SILK, SparkFun-Jumpers:JUMPER-SMT_3_1-NC_TRACE_SILK
- added R1, R2: 5.1K, SparkFun-Resistors:RESISTOR0402
- added R4: 50k, SparkFun-Resistors:RESISTOR0402
- added U10: W25N01GVZEIG_TR, W25N01GVZEIG_TR:W25N01GVZEIG_TR
- C17: value 10uF -> 0.01uF; device SparkFun-Capacitors:10UF-POLAR-0603-6.3V-20%(TANT) -> SparkFun-Capacitors:CAP-0402
- C23: value 0.uF -> 4.7uF
- R25: value (none) -> 4K
- R5: value (none) -> 50k
Connections:
- net RX renamed SERCOM3_RX
- net TX renamed SERCOM3_TX
- removed net SERCOM7_RX: U4.TX, U6.PB31
- removed net SERCOM7_TX: U4.RX, U6.PB30
- new net BAT_OK: JP2.3, U9.VBAT_OK
- new net N$4: J4.CC2, R1.2
- new net N$5: J4.CC1, R2.2
- new net N$6: JP2.2, U2.EN
- new net SERCOM1_RX: U4.TX, U6.PA01
- new net SERCOM1_TX: U4.RX, U6.PA00
- net !RESET: now also R4.1, U$2.S; no longer R5.2, U$2.D
- net BUTTON: now also R5.1, U$2.D, U6.PA27; no longer U$2.S
- net CS_MEM: now also U10./CS; no longer U7.!CS
- net D+: now also J4.D+; no longer J2.D+
- net D-: now also J4.D-; no longer J2.D-
- net GND: now also C17.1, C19.-, J4.GND, JP3.GNDDTCT, R1.1, R2.1, U$3.1, U10.GND; no longer C17.-, R5.1, U7.GND
- net GPS_INT: now also U6.PA02; no longer U6.PA00
- net LED: now also U6.PA16; no longer U6.PB16
- net N$14: now also U10.VCC; no longer U7.VCC
- net N$3: now also C17.2
- net SERCOM5_MISO: now also U10.DO(IO1); no longer U7.SO(I/O1)
- net SERCOM5_MOSI: now also U10.DI(IO0); no longer U7.SI(I/O0)
- net SERCOM5_SCK: now also U10.CLK; no longer U7.SCK
- net VBUS: now also J4.VBUS; no longer J2.VBUS
- net VCC-ISO: now also R4.2, R5.2; no longer U$3.1
- net VCC_1: now also C19.+, U10./HOLD(IO3), U10./WP(IO2); no longer C17.+, U7.!HOLD!/!RESET!(I/O3), U7.!WP!(I/O2)
- net VIN: now also JP2.1; no longer U2.EN
Other:
- moved on the sheet: C2, R5
