File: Parabeep V0.3/rewire/ParaBeep V0.3_2.brd (EAGLE design)
At the start: 35.3 x 57.5 mm, 65 parts, among them IC2 MCP73811/2, Q1 500mA/300V, U1 ADXL345, U2 TPS78330DDCRDDC5_TEX-L, U3 TPS78330DDCRDDC5_TEX-L, U4 UBLOX_SAM_M8Q-0-10, U5 MS5803-14BA, U6 ATSAMD51J20A-A, U7 AT25SF128A-SHB-T, U8 RN4871-V/RM118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

Commit message: bluetooth working, usb next
Parts:
- added R1: 10k, SparkFun-Resistors:0402
- R5: value (none) -> 10k
- moved R5 1.49 mm to (22.0, 13.6), turned to 0 degrees
Connections:
- net !RESET: now also R5.1, U$2.2; no longer R5.2, U$2.3
- net BUTTON: now also R1.1, U$2.3; no longer U$2.2
- net GND: now also U$3.P$1; no longer R5.1
- net VCC-ISO: now also R1.2, R5.2; no longer U$3.P$1
Routing:
- net !RESET: track 22.2 -> 25.7 mm, vias 2 -> 3
- net BUTTON: track 2.49 -> 5.41 mm
- net VCC-ISO: track 74.3 -> 71.6 mm
- net GND: vias 72 -> 71
